File: es/electric/serie-paralelo/electric-serie-paralelo-2.sch (KiCad schematic (older format))
At the start: 61 parts

Commit message: Actualizado con pequeños cambios.
Connections:
- net at L58.~, L62.~: now also V.~
- net at V.~: now also L63.~; no longer L59.~
- net at L63.~: now also L59.~; no longer V.~
- net at L76.~, L80.~: no longer V.~
- net at L74.~, L78.~: now also V.~
- net at L42.~, L48.~: now also V.~
- net at L47.~, V.~: no longer L43.~
- net at L45.~, V.~: now also L44.~
- net at L50.~, L54.~: now also V.~
- new net: L51.~, L55.~, V.~
- new net: L57.~, L61.~, V.~
- new net: L58.~, L62.~
- new net: L59.~, V.~
- new net: L60.~, L64.~, V.~
- new net: L65.~, L70.~, V.~
- new net: L68.~, L69.~, V.~
- new net: L66.~, L71.~, V.~
- new net: L67.~, L72.~, V.~
- new net: L76.~, L80.~, V.~
- new net: L74.~, L78.~
- new net: L75.~, L79.~, V.~
- new net: L42.~, L48.~
- new net: L43.~, L47.~, V.~
- new net: L45.~, V.~
- new net: L50.~, L54.~
- new net: L49.~, L53.~, V.~
- new net: L52.~, L56.~, V.~
- new net: L41.~, L46.~, V.~
Changed lines of the file:
@@
 EESchema Schematic File Version 4
-LIBS:electric-serie-paralelo-cache
-EELAYER 26 0
+EELAYER 30 0
 EELAYER END
 $Descr A4 8268 11693 portrait
