File: es/electric/electric-cableado/electric-cableado-3.sch (KiCad schematic (older format))
At the start: 115 parts, among them Q1 NPN

Commit message: Nuevos circuitos para cablear
Parts:
- removed CP?: CopyRight, symbol simbolos:CopyRight
- added CP?: CopyRight, symbol simbolos:CopyRight
Connections:
- net at S1.~: now also R1.~; no longer V1.~
- net at R1.~: now also D1.~; no longer S1.~
- net at R1.~: now also R2.~, V1.~; no longer Q1.~
- net at V1.~: now also D1.~, D2.~; no longer S1.~
- net at V1.~: now also C1.~, D1.~; no longer S1.~
- net at R3.~: now also D1.~; no longer Q1.~
- net at D1.~: now also R1.~, V1.~; no longer R3.~
- net at Q1.~, R2.~: now also V1.~; no longer R1.~
- net at S1.~: now also R2.~; no longer R1.~
- net at R2.~: now also D2.~; no longer S1.~
- new net: S1.~, V1.~ (x3)
- new net: Q1.~, R1.~
- new net: Q1.~, R1.~, V1.~
- new net: Q1.~, R3.~
- new net: Q1.~, R1.~, R2.~
- new net: R1.~, S1.~
Changed lines of the file:
@@
-	1    0    0    -1
-$EndComp
-$Comp
-L simbolos:CopyRight CP?
-U 1 1 5BC453A4
-P 3900 11400
-F 0 "CP?" H 4325 11725 40  0001 C CNN
-F 1 "CopyRight" H 4075 11725 40  0001 C CNN
-F 2 "" H 3800 11750 50  0001 C CNN
-F 3 "" H 3900 11600 50  0001 C CNN
-F 4 "CC BY-SA 4.0" H 3575 11350 50  0000 C CNN "License"
-F 5 "" H 4450 11350 50  0000 C CNN "Author"
-F 6 "" H 4025 11350 50  0000 C CNN "Date"
-F 7 "www.picuino.com" H 4275 11350 50  0000 C CNN "Web"
-	1    3900 11400
 	1    0    0    -1
 $EndComp
@@
 Wire Wire Line
 	7500 8900 7500 9000
+$Comp
+L simbolos:CopyRight CP?
+U 1 1 60A48BBB
+P 3825 200
+F 0 "CP?" H 4250 525 40  0001 C CNN
+F 1 "CopyRight" H 4000 525 40  0001 C CNN
+F 2 "" H 3725 550 50  0001 C CNN
+F 3 "" H 3825 400 50  0001 C CNN
+F 4 "CC BY-SA 4.0" H 3375 125 75  0000 C CNN "License"
+F 5 "" H 4375 150 50  0000 C CNN "Author"
+F 6 "" H 3950 150 50  0000 C CNN "Date"
+F 7 "www.picuino.com" H 4350 125 75  0000 C CNN "Web"
+	1    3825 200
+	1    0    0    -1
+$EndComp
 $EndSCHEMATC
