File: es/electric/electric-cableado/electric-cableado.sch (KiCad schematic (older format))
At the start: 100 parts

Commit message: Nuevos circuitos para cablear
Connections:
- net at S1.~: now also L1.~; no longer V1.~
- net at L1.~: now also V1.~; no longer S1.~
- net at V1.~: now also S1.~; no longer L2.~
- net at S1.~: now also S2.~; no longer V1.~
- net at S1.~, S2.~: now also L1.~, L2.~; no longer V1.~
- net at V1.~: now also L1.~, L2.~; no longer S1.~
- net at L1.~, L2.~: now also S2.~; no longer V1.~
- new net: S1.~, V1.~ (x2)
- new net: L2.~, V1.~
- new net: S1.~, S2.~, V1.~ (x2)
- new net: L1.~, L2.~, V1.~
- new net: S1.~, S2.~
Changed lines of the file:
@@
 L simbolos:CopyRight CP?
 U 1 1 5BC453A4
-P 3900 11400
-F 0 "CP?" H 4325 11725 40  0001 C CNN
-F 1 "CopyRight" H 4075 11725 40  0001 C CNN
-F 2 "" H 3800 11750 50  0001 C CNN
-F 3 "" H 3900 11600 50  0001 C CNN
-F 4 "CC BY-SA 4.0" H 3575 11350 50  0000 C CNN "License"
-F 5 "" H 4450 11350 50  0000 C CNN "Author"
-F 6 "" H 4025 11350 50  0000 C CNN "Date"
-F 7 "www.picuino.com" H 4275 11350 50  0000 C CNN "Web"
-	1    3900 11400
+P 4200 200
+F 0 "CP?" H 4625 525 40  0001 C CNN
+F 1 "CopyRight" H 4375 525 40  0001 C CNN
+F 2 "" H 4100 550 50  0001 C CNN
+F 3 "" H 4200 400 50  0001 C CNN
+F 4 "CC BY-SA 4.0" H 3750 125 75  0000 C CNN "License"
+F 5 "" H 4750 150 50  0000 C CNN "Author"
+F 6 "" H 4325 150 50  0000 C CNN "Date"
+F 7 "www.picuino.com" H 4725 125 75  0000 C CNN "Web"
+	1    4200 200
 	1    0    0    -1
 $EndComp
