File: es/electric/bornas-1/electric-bornas-conmutador.sch (KiCad schematic (older format))
At the start: 16 parts, among them X1 borna_12x2

Commit message: Cambios a 19/09/2021
Other:
- note added: "1 x CONMUTADOR DE\n 1 CIRCUITO\n 2 POSICIONES"
- note removed: "2 x CONMUTADOR DE\n 1 CIRCUITO\n 2 POSICIONES"
Changed lines of the file:
@@
 EESchema Schematic File Version 4
-EELAYER 26 0
+EELAYER 30 0
 EELAYER END
 $Descr A4 8268 11693 portrait
@@
 	4050 6500 5050 6500
 Text Notes 1650 6850 0    100  ~ 0
-2 x CONMUTADOR DE\n    1 CIRCUITO\n    2 POSICIONES
+1 x CONMUTADOR DE\n    1 CIRCUITO\n    2 POSICIONES
 Text Notes 1650 5800 0    100  ~ 0
 1 x PILA DE PETACA
@@
 	5000 10500 4700 10500
 Wire Wire Line
-	4700 10300 5300 10300
-Wire Wire Line
-	5300 10300 5300 8900
-Wire Wire Line
-	5300 8900 4700 8900
-Wire Wire Line
-	4700 10700 5600 10700
-Wire Wire Line
-	5600 10700 5600 10100
-Wire Wire Line
-	5600 10100 4700 10100
+	4700 10300 5250 10300
+Wire Wire Line
+	5250 10300 5250 8900
+Wire Wire Line
+	5250 8900 4700 8900
+Wire Wire Line
+	4700 10700 5500 10700
+Wire Wire Line
+	5500 10700 5500 10100
+Wire Wire Line
+	5500 10100 4700 10100
 Wire Wire Line
 	4700 10100 4900 10000
 Wire Wire Line
-	4900 10000 5600 10000
-Wire Wire Line
-	5600 10000 5600 8700
-Wire Wire Line
-	5600 8700 4700 8700
+	4900 10000 5500 10000
+Wire Wire Line
+	5500 10000 5500 8700
+Wire Wire Line
+	5500 8700 4700 8700
 Connection ~ 4700 10100
 $EndSCHEMATC
