File: es/electric/bornas-1/electric-bornas-conmutador-doble.kicad_sch (KiCad schematic)
At the start: 16 parts

Commit message: Trasladar proyectos KiCAD 5 a KiCAD 6. Thickness 12mils
Parts:
- CP1: value (none) -> CopyRight
- L1: value (none) -> lampara
- L1, L2, L?: value (none) -> lampara_pack
- S1, S2, S?: value (none) -> selector_pack
- S1, S2, S?: value (none) -> conmutador
- V1, V?: value (none) -> pila_petaca
- V1: value (none) -> Pila
- X1: value (none) -> borna_12x2
- X?: value (none) -> borna_6x2
Connections:
- net at X1.: now also S2.
- net at V1.: now also S1.; no longer L1.
- net at S1.: now also S2.; no longer V1.
- new net: V1., X1.
- new net: L1., X1.
- new net: L2., X1.
- new net: S1., X1. (x2)
- new net: S2., X1. (x2)
- new net: L1., V1.
- new net: S1., S2.
Changed lines of the file:
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@@
       (effects (font (size 1.016 1.016)) hide)
     )
-    (property "Value" "" (id 1) (at 100.965 281.305 0)
+    (property "Value" "CopyRight" (id 1) (at 100.965 281.305 0)
       (effects (font (size 1.016 1.016)) hide)
     )
@@
       (effects (font (size 2.54 2.54)))
     )
-    (property "Value" "" (id 1) (at 115.57 214.63 0)
+    (property "Value" "borna_12x2" (id 1) (at 115.57 214.63 0)
       (effects (font (size 1.27 1.27)) hide)
     )
@@
       (effects (font (size 1.27 1.27)) hide)
     )
-    (pin "~")
-    (pin "~")
-    (pin "~")
-    (pin "~")
-    (pin "~")
-    (pin "~")
-    (pin "~")
-    (pin "~")
-    (pin "~")
-    (pin "~")
-    (pin "~")
-    (pin "~")
-    (pin "~")
-    (pin "~")
-    (pin "~")
-    (pin "~")
-    (pin "~")
-    (pin "~")
-    (pin "~")
-    (pin "~")
-    (pin "~")
-    (pin "~")
-    (pin "~")
-    (pin "~")
+    (pin "")
+    (pin "")
+    (pin "")
+    (pin "")
+    (pin "")
+    (pin "")
+    (pin "")
+    (pin "")
+    (pin "")
+    (pin "")
+    (pin "")
+    (pin "")
+    (pin "")
+    (pin "")
+    (pin "")
+    (pin "")
+    (pin "")
+    (pin "")
+    (pin "")
+    (pin "")
+    (pin "")
+    (pin "")
+    (pin "")
+    (pin "")
   )
   (symbol (lib_id "simbolos:pila_petaca") (at 99.06 220.98 270) (mirror x) (unit 1)
@@
       (effects (font (size 2.54 2.54)) (justify left))
     )
-    (property "Value" "" (id 1) (at 90.805 217.17 0)
+    (property "Value" "pila_petaca" (id 1) (at 90.805 217.17 0)
       (effects (font (size 1.27 1.27)) hide)
     )
@@
       (effects (font (size 2.54 2.54)))
     )
-    (pin "~")
-    (pin "~")
+    (pin "")
+    (pin "")
   )
   (symbol (lib_id "simbolos:pila_petaca") (at 22.86 137.16 0) (unit 1)
@@
       (effects (font (size 2.54 2.54)) (justify left) hide)
     )
-    (property "Value" "" (id 1) (at 26.67 145.415 0)
+    (property "Value" "pila_petaca" (id 1) (at 26.67 145.415 0)
       (effects (font (size 1.27 1.27)) hide)
     )
@@
       (effects (font (size 2.54 2.54)))
     )
-    (pin "~")
-    (pin "~")
+    (pin "")
+    (pin "")
   )
   (symbol (lib_id "simbolos:Pila") (at 15.24 48.26 0) (unit 1)
@@
       (effects (font (size 2.54 2.54)) (justify left))
     )
-    (property "Value" "" (id 1) (at 17.78 50.165 0)
+    (property "Value" "Pila" (id 1) (at 17.78 50.165 0)
       (effects (font (size 1.27 1.27)) hide)
     )
@@
       (effects (font (size 1.27 1.27)) hide)
     )
-    (pin "~")
-    (pin "~")
+    (pin "")
+    (pin "")
   )
   (symbol (lib_id "simbolos:lampara") (at 83.82 50.8 0) (unit 1)
@@
       (effects (font (size 2.54 2.54)) (justify left))
     )
-    (property "Value" "" (id 1) (at 85.09 64.135 90)
+    (property "Value" "lampara" (id 1) (at 85.09 64.135 90)
       (effects (font (size 1.27 1.27)) hide)
     )
@@
       (effects (font (size 1.27 1.27)) hide)
     )
-    (pin "~")
-    (pin "~")
+    (pin "")
+    (pin "")
   )
   (symbol (lib_id "simbolos:lampara_pack") (at 50.8 274.32 0) (unit 1)
@@
       (effects (font (size 2.54 2.54)))
     )
-    (property "Value" "" (id 1) (at 63.5 276.225 0)
+    (property "Value" "lampara_pack" (id 1) (at 63.5 276.225 0)
       (effects (font (size 1.27 1.27)) hide)
     )
@@
       (effects (font (size 1.27 1.27)) hide)
     )
-    (pin "~")
-    (pin "~")
+    (pin "")
+    (pin "")
   )
   (symbol (lib_id "simbolos:lampara_pack") (at 12.7 274.32 0) (unit 1)
@@
       (effects (font (size 2.54 2.54)))
     )
-    (property "Value" "" (id 1) (at 25.4 276.225 0)
+    (property "Value" "lampara_pack" (id 1) (at 25.4 276.225 0)
       (effects (font (size 1.27 1.27)) hide)
     )
@@
       (effects (font (size 1.27 1.27)) hide)
     )
-    (pin "~")
-    (pin "~")
+    (pin "")
+    (pin "")
   )
   (symbol (lib_id "simbolos:borna_6x2") (at 128.27 177.8 270) (unit 1)
@@
       (effects (font (size 2.54 2.54)) (justify right) hide)
     )
-    (property "Value" "" (id 1) (at 129.54 181.61 0)
+    (property "Value" "borna_6x2" (id 1) (at 129.54 181.61 0)
       (effects (font (size 1.27 1.27)) hide)
     )
@@
       (effects (font (size 1.27 1.27)) hide)
     )
-    (pin "~")
-    (pin "~")
-    (pin "~")
-    (pin "~")
-    (pin "~")
-    (pin "~")
-    (pin "~")
-    (pin "~")
-    (pin "~")
-    (pin "~")
-    (pin "~")
-    (pin "~")
+    (pin "")
+    (pin "")
+    (pin "")
+    (pin "")
+    (pin "")
+    (pin "")
+    (pin "")
+    (pin "")
+    (pin "")
+    (pin "")
+    (pin "")
+    (pin "")
   )
   (symbol (lib_id "simbolos:conmutador") (at 20.32 184.15 0) (unit 1)
@@
       (effects (font (size 2.54 2.54)) hide)
     )
-    (property "Value" "" (id 1) (at 20.32 185.42 0)
+    (property "Value" "conmutador" (id 1) (at 20.32 185.42 0)
       (effects (font (size 1.27 1.27)) hide)
     )
@@
       (effects (font (size 1.27 1.27)) hide)
     )
-    (pin "~")
-    (pin "~")
-    (pin "~")
+    (pin "")
+    (pin "")
+    (pin "")
   )
   (symbol (lib_id "simbolos:selector_pack") (at 53.34 223.52 0) (unit 1)
@@
       (effects (font (size 2.54 2.54)) (justify left))
     )
-    (property "Value" "" (id 1) (at 58.42 218.44 0)
+    (property "Value" "selector_pack" (id 1) (at 58.42 218.44 0)
       (effects (font (size 1.27 1.27)) hide)
     )
@@
       (effects (font (size 1.27 1.27)) hide)
     )
-    (pin "~")
-    (pin "~")
-    (pin "~")
+    (pin "")
+    (pin "")
+    (pin "")
   )
   (symbol (lib_id "simbolos:selector_pack") (at 17.78 223.52 0) (unit 1)
@@
       (effects (font (size 2.54 2.54)) (justify left))
     )
-    (property "Value" "" (id 1) (at 22.86 218.44 0)
+    (property "Value" "selector_pack" (id 1) (at 22.86 218.44 0)
       (effects (font (size 1.27 1.27)) hide)
     )
@@
       (effects (font (size 1.27 1.27)) hide)
     )
-    (pin "~")
-    (pin "~")
-    (pin "~")
+    (pin "")
+    (pin "")
+    (pin "")
   )
   (symbol (lib_id "simbolos:conmutador") (at 30.48 38.1 0) (unit 1)
@@
       (effects (font (size 2.54 2.54)))
     )
-    (property "Value" "" (id 1) (at 30.48 39.37 0)
+    (property "Value" "conmutador" (id 1) (at 30.48 39.37 0)
       (effects (font (size 1.27 1.27)) hide)
     )
@@
       (effects (font (size 1.27 1.27)) hide)
     )
-    (pin "~")
-    (pin "~")
-    (pin "~")
+    (pin "")
+    (pin "")
+    (pin "")
   )
   (symbol (lib_id "simbolos:selector_pack") (at 21.59 170.18 0) (unit 1)
@@
       (effects (font (size 2.54 2.54)) (justify left) hide)
     )
-    (property "Value" "" (id 1) (at 26.67 165.1 0)
+    (property "Value" "selector_pack" (id 1) (at 26.67 165.1 0)
       (effects (font (size 1.27 1.27)) hide)
     )
@@
       (effects (font (size 1.27 1.27)) hide)
     )
-    (pin "~")
-    (pin "~")
-    (pin "~")
+    (pin "")
+    (pin "")
+    (pin "")
   )
   (symbol (lib_id "simbolos:lampara_pack") (at 102.87 151.13 0) (unit 1)
@@
       (effects (font (size 2.54 2.54)) hide)
     )
-    (property "Value" "" (id 1) (at 115.57 153.035 0)
+    (property "Value" "lampara_pack" (id 1) (at 115.57 153.035 0)
       (effects (font (size 1.27 1.27)) hide)
     )
@@
       (effects (font (size 1.27 1.27)) hide)
     )
-    (pin "~")
-    (pin "~")
+    (pin "")
+    (pin "")
   )
   (symbol (lib_id "simbolos:conmutador") (at 71.12 38.1 0) (mirror y) (unit 1)
@@
       (effects (font (size 2.54 2.54)))
     )
-    (property "Value" "" (id 1) (at 71.12 39.37 0)
+    (property "Value" "conmutador" (id 1) (at 71.12 39.37 0)
       (effects (font (size 1.27 1.27)) hide)
     )
@@
       (effects (font (size 1.27 1.27)) hide)
     )
-    (pin "~")
-    (pin "~")
-    (pin "~")
+    (pin "")
+    (pin "")
+    (pin "")
   )
   (sheet (at 218.44 29.21) (size 66.04 7.62) (fields_autoplaced)
