File: es/electric/pcb-luces-led-navidad/pcb-luces-led-navidad.sch (KiCad schematic (older format))
At the start: 22 parts, among them SW1 SW_SPDT, U1 74HC14

Commit message: Cambios a 16/01/2022
Parts:
- SW1: footprint pcb-luces-led-navidad:SPDT -> Button_Switch_THT:SW_Slide_1P2T_CK_OS102011MS2Q
Changed lines of the file:
@@
 F 0 "SW1" H 7375 2291 50  0000 C CNN
 F 1 "SW_SPDT" H 7375 2198 50  0000 C CNN
-F 2 "pcb-luces-led-navidad:SPDT" H 7375 2000 50  0001 C CNN
+F 2 "Button_Switch_THT:SW_Slide_1P2T_CK_OS102011MS2Q" H 7375 2000 50  0001 C CNN
 F 3 "~" H 7375 2000 50  0001 C CNN
 	1    7375 2000
