File: es/electric/pcb-luces-led-navidad/pcb-luces-led-navidad.kicad_pcb (KiCad board)
At the start: 2 copper layers, 59.7 x 39.4 mm, 24 parts, among them SW1 SW_SPDT, U1 74HC14

Commit message: Cambios a 16/01/2022
Parts:
- removed the Picuino_Logo_B6 at (69.8, 87.6)
- added M3: , pcb-luces-led-navidad:SCREW_M3, F.Cu at (54.0, 87.0)
- added M3: , pcb-luces-led-navidad:SCREW_M3, F.Cu at (54.0, 54.0)
- added M3: , pcb-luces-led-navidad:SCREW_M3, F.Cu at (107.3, 87.0)
- added M3: , pcb-luces-led-navidad:SCREW_M3, F.Cu at (107.3, 54.0)
- SW1: footprint pcb-luces-led-navidad:SPDT -> Button_Switch_THT:SW_Slide_1P2T_CK_OS102011MS2Q
- moved C2 6.35 mm to (65.4, 85.1)
- moved C1 6.35 mm to (59.7, 85.1)
- moved SW1 3.24 mm to (65.4, 53.3)
- moved C3 0.09 mm to (59.7, 62.9), turned to 0 degrees
Routing:
- net GND: track 59.4 -> 56.4 mm
- net Net-(BT1-Pad1): track 11.8 -> 14.0 mm
- net Net-(C3-Pad1): track 27.3 -> 29.2 mm
- net Net-(C1-Pad1): track 32.7 -> 34.5 mm
- net +BATT: track 119.8 -> 121.5 mm
Other:
- board text added: "+"
- board text added: "-"
- board text added: "2022-R2"
- board text removed: "2022-R1"

Commit message: Cambios a 20/01/2022
Parts:
- added Picuino_Logo_B6: VAL**, pcb-luces-led-navidad:Picuino_Logo_B6, B.Cu at (103.5, 69.8)
- C1, C2, C3: footprint Capacitor_THT:CP_Radial_D5.0mm_P2.00mm -> pcb-luces-led-navidad:CP_Radial_D5.0mm_P2.00mm
- R2, R3, R4, R5, R6, R7, R8, R9: footprint Resistor_THT:R_Axial_DIN0411_L9.9mm_D3.6mm_P12.70mm_Horizontal -> pcb-luces-led-navidad:R_Axial_DIN0411_L9.9mm_D3.6mm_P12.70mm_Horizontal
- moved Picuino_Logo_B6 0.64 mm to (88.9, 70.5)

Commit message: Versión r2
Parts:
- moved SW1 1.66 mm to (66.5, 54.6)
Routing:
- net +BATT: track 121.5 -> 135.2 mm
- net GND: track 56.4 -> 59.0 mm
- net Net-(BT1-Pad1): track 14.0 -> 14.7 mm
