File: es/neumatic/simbolos/neumatic-simbolos-nombres.sch (KiCad schematic (older format))
At the start: 45 parts

Commit message: Cambios a 19/05/2022
Parts:
- removed M?: Marco_1, symbol simbolos:Marco_1
- added M? (x30): Marco_1, symbol simbolos:Marco_1
- added M? (x3): Marco_2, symbol simbolos:Marco_2
- added V?: Manometro, symbol simbolos:Manometro
- added V?: Calderin, symbol simbolos:Calderin
- added V?: Fuente_presion, symbol simbolos:Fuente_presion
- added V?: Piston_simple_efecto, symbol simbolos:Piston_simple_efecto
- added V?: Piston_doble_efecto, symbol simbolos:Piston_doble_efecto
- added V?: Valvula_antirretorno, symbol simbolos:Valvula_antirretorno
- added V?: Estrangulador, symbol simbolos:Estrangulador
- added V?: Valvula_simultaneidad, symbol simbolos:Valvula_simultaneidad
- added V?: Valvula_or, symbol simbolos:Valvula_or
Other:
- note added: "DEPÓSITO"
- note added: "ESTRANGULADOR"
- note added: "FUENTE DE\nPRESIÓN"
- note added: "MANÓMETRO"
- note added: "PISTON DE \nDOBLE EFECTO"
- note added: "PISTON DE \nSIMPLE EFECTO"
- note added: "VÁLVULA DE\nSIMULTANEIDAD"
- note added: "VÁLVULA OR"
- note added: "VÁLVULA\nANTIRRETORNO"
