File: es/neumatic/simbolos-nombres/neumatic-nombres.sch (KiCad schematic (older format))
At the start: 42 parts

Commit message: Cambios a 23/05/2022.
Other:
- note added: "ESCAPE\nDE AIRE"
- note removed: "ESCAPE\nRÁPIDO"
Changed lines of the file:
@@
 $EndComp
 Text Notes 6875 7800 0    100  ~ 0
-ESCAPE\nRÁPIDO
+ESCAPE\nDE AIRE
 $Comp
 L simbolos:Marco_1 M?
