File: es/neumatic/simbolos-nombres/neumatic-simbolos-nombres.sch (KiCad schematic (older format))
At the start: 83 parts

Commit message: Cambios a 23/05/2022.
Other:
- note added: "ESCAPE\nDE AIRE"
- note removed: "ESCAPE\nRÁPIDO"
Changed lines of the file:
@@
-	1    0    0    -1
-$EndComp
-Text Notes 6875 7800 0    100  ~ 0
-ESCAPE\nRÁPIDO
-$Comp
-L simbolos:Marco_1 M?
-U 1 1 6289B160
-P 5500 7350
-F 0 "M?" H 5625 7175 100 0001 C CNN
-F 1 "Marco_1" H 5650 7300 50  0001 C CNN
-F 2 "" H 5550 7200 50  0001 C CNN
-F 3 "" H 5550 7200 50  0001 C CNN
-	1    5500 7350
 	1    0    0    -1
 $EndComp
@@
 	1    0    0    -1
 $EndComp
+$Comp
+L simbolos:Marco_1 M?
+U 1 1 6289B160
+P 5500 7350
+F 0 "M?" H 5625 7175 100 0001 C CNN
+F 1 "Marco_1" H 5650 7300 50  0001 C CNN
+F 2 "" H 5550 7200 50  0001 C CNN
+F 3 "" H 5550 7200 50  0001 C CNN
+	1    5500 7350
+	1    0    0    -1
+$EndComp
+Text Notes 6875 7800 0    100  ~ 0
+ESCAPE\nDE AIRE
 $EndSCHEMATC

Commit message: Cambios a 28/05/2022.
Parts:
- removed V?: Estrangulador, symbol simbolos:Estrangulador
- removed V?: Valvula_antirretorno, symbol simbolos:Valvula_antirretorno
- added V?: Estrangulador_unidireccional, symbol simbolos:Estrangulador_unidireccional
- V?: value Escape_rápido -> Escape; symbol simbolos:Escape_rápido -> simbolos:Escape
Connections:
- wire segments 6 -> 0
Changed lines of the file:
@@
-$EndComp
-$Comp
-L simbolos:Estrangulador V?
-U 1 1 62882C39
-P 6150 6000
-F 0 "V?" H 6100 5850 100 0001 L CNN
-F 1 "Estrangulador" H 6150 6125 50  0001 C CNN
-F 2 "" H 6150 5875 50  0001 C CNN
-F 3 "" H 6150 5875 50  0001 C CNN
-	1    6150 6000
-	1    0    0    -1
-$EndComp
-$Comp
-L simbolos:Valvula_antirretorno V?
-U 1 1 62882F63
-P 6150 5700
-F 0 "V?" H 6100 5550 100 0001 L CNN
-F 1 "Valvula_antirretorno" H 6150 5825 50  0001 C CNN
-F 2 "" H 6150 5575 50  0001 C CNN
-F 3 "" H 6150 5575 50  0001 C CNN
-	1    6150 5700
-	-1   0    0    1
 $EndComp
 $Comp
@@
 	1    0    0    -1
 $EndComp
-Wire Wire Line
-	6300 5700 6325 5700
-Wire Wire Line
-	6325 5700 6325 6000
-Wire Wire Line
-	6325 6000 6425 6000
-Connection ~ 6325 6000
-Wire Wire Line
-	6000 5700 5975 5700
-Wire Wire Line
-	5975 5700 5975 6000
-Wire Wire Line
-	5975 6000 5875 6000
-Connection ~ 5975 6000
 Wire Notes Line
 	8100 11500 8100 300
@@
 PILOTAJE CON\nENCLAVAMIENTO
 $Comp
-L simbolos:Escape_rápido V?
+L simbolos:Escape V?
 U 1 1 62897B4E
 P 6150 7575
 F 0 "V?" H 6025 7550 100 0001 L CNN
-F 1 "Escape_rápido" H 6175 7875 50  0001 C CNN
+F 1 "Escape" H 6175 7875 50  0001 C CNN
 F 2 "" H 6150 7450 50  0001 C CNN
 F 3 "" H 6150 7450 50  0001 C CNN
@@
 Text Notes 6875 7800 0    100  ~ 0
 ESCAPE\nDE AIRE
+$Comp
+L simbolos:Estrangulador_unidireccional V?
+U 1 1 6291FFE3
+P 6150 5750
+F 0 "V?" H 6100 5575 100 0001 L CNN
+F 1 "Estrangulador_unidireccional" H 6150 5465 50  0001 C CNN
+F 2 "" H 6150 5625 50  0001 C CNN
+F 3 "" H 6150 5625 50  0001 C CNN
+	1    6150 5750
+	1    0    0    -1
+$EndComp
 $EndSCHEMATC
