File: es/neumatic/simbolos-nombres/neumatic-simbolos.sch (KiCad schematic (older format))
At the start: 83 parts

Commit message: Cambios a 28/05/2022.
Parts:
- V?: value Escape_rápido -> Escape; symbol simbolos:Escape_rápido -> simbolos:Escape
Changed lines of the file:
@@
 $EndComp
 $Comp
-L simbolos:Escape_rápido V?
+L simbolos:Escape V?
 U 1 1 628A62E7
 P 6150 7575
 F 0 "V?" H 6025 7550 100 0001 L CNN
-F 1 "Escape_rápido" H 6175 7875 50  0001 C CNN
+F 1 "Escape" H 6175 7875 50  0001 C CNN
 F 2 "" H 6150 7450 50  0001 C CNN
 F 3 "" H 6150 7450 50  0001 C CNN
