File: es/electric/simbolos-nombres/electric-nombres.kicad_sch (KiCad schematic)
At the start: 49 parts

Commit message: Cambios a 07/10/2022
Other:
- note added: "POTENCIÓMETRO"
- note removed: "RESISTENCIA VARIABLE"
Changed lines of the file:
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@@
+    (effects (font (size 2.54 2.54)) (justify left bottom))
+  )
+  (text "POTENCIÓMETRO" (at 173.99 120.015 0)
     (effects (font (size 2.54 2.54)) (justify left bottom))
   )
@@
     (effects (font (size 2.54 2.54)) (justify left bottom))
   )
-  (text "RESISTENCIA\nVARIABLE" (at 174.625 121.92 0)
-    (effects (font (size 2.54 2.54)) (justify left bottom))
-  )
