File: es/electric/simbolos-nombres/electric-simbolos-nombres.kicad_sch (KiCad schematic)
At the start: 87 parts, among them J1 conector, K1 CONTACTO, K1 RELE, M1 MOTOR, Q1 TRANSISTOR, Q2 TRANSISTOR, U1 AO, U1 logic_and, U2 logic_and, U3 logic_and, U4 logic_and, U5 logic_and, U6 logic_and

Commit message: Cambios a 07/10/2022
Parts:
- removed R3: RESISTENCIA, symbol electric-simbolos-nombres-rescue:resistencia_variable-simbolos
- added R2: potenciometro, symbol simbolos-electricos:potenciometro
- Q1: symbol electric-simbolos-nombres-rescue:NPN-simbolos -> simbolos-electricos:NPN
- Q2: symbol electric-simbolos-nombres-rescue:PNP-simbolos -> simbolos-electricos:PNP
- R3: renamed from R1; symbol electric-simbolos-nombres-rescue:NTC-simbolos -> simbolos-electricos:NTC
- R4: renamed from R2; symbol electric-simbolos-nombres-rescue:LDR-simbolos -> simbolos-electricos:LDR
- TR1: symbol electric-simbolos-nombres-rescue:transformador-simbolos -> simbolos-electricos:transformador
- V: symbol electric-simbolos-nombres-rescue:voltimetro-simbolos -> simbolos-electricos:voltimetro
- V1: symbol electric-simbolos-nombres-rescue:Pila-simbolos -> simbolos-electricos:Pila
- V?: symbol electric-simbolos-nombres-rescue:tierra-simbolos -> simbolos-electricos:tierra
- Z1: symbol electric-simbolos-nombres-rescue:zumbador-simbolos -> simbolos-electricos:zumbador
- Z2: symbol electric-simbolos-nombres-rescue:altavoz-simbolos -> simbolos-electricos:altavoz
- renumbered S4 to S2, S2 to S3, S3 to S4
Other:
- note added: "POTENCIÓMETRO"
- note removed: "RESISTENCIA VARIABLE"
