File: source/neumatic/circuitos-neumaticos/neumatic-circuitos.kicad_sch (KiCad schematic)
At the start: 47 parts

Commit message: 10/04/2024 Update
Parts:
- added V1, V2: Valvula_antirretorno, symbol neumatic-simbolos-nombres-rescue:Valvula_antirretorno-simbolos
Connections:
- net at V?.: now also V?.; no longer V?. (x2)
- net at V?.: now also V?. (x5)
- new net: V?., V?. (x2)
- new net: V?., V?., V?., V?.
