File: source/neumatic/simbolos-nombres/neumatic-simbolos-nombres.kicad_sch (KiCad schematic)
At the start: 82 parts

Commit message: 10/04/2024 Update
Other:
- note added: "DEPÓSITO O CALDERÍN"
- note added: "VÁLVULA DE SIMULTANEIDAD AND"
- note added: "VÁLVULA SELECTORA OR"
- note removed: "DEPÓSITO"
- note removed: "VÁLVULA DE SIMULTANEIDAD"
- note removed: "VÁLVULA OR"
