File: source/electric/simbolos-nombres/electric-nombres.kicad_sch (KiCad schematic)
At the start: 49 parts

Commit message: 31/05/2024 Update
Other:
- note added: "ALTERNADOR"
- note removed: "GENERADOR"
Changed lines of the file:
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@@
     (effects (font (size 2.54 2.54)) (justify left bottom))
   )
-  (text "GENERADOR" (at 40.005 43.815 0)
+  (text "ALTERNADOR" (at 40.005 43.815 0)
     (effects (font (size 2.54 2.54)) (justify left bottom))
   )
