File: source/electric/simbolos-nombres/electric-simbolos-nombres.kicad_sch (KiCad schematic)
At the start: 87 parts, among them J1 conector, K1 CONTACTO, K1 RELE, M1 MOTOR, Q1 TRANSISTOR, Q2 TRANSISTOR, U1 AO, U1 logic_and, U2 logic_and, U3 logic_and, U4 logic_and, U5 logic_and, U6 logic_and

Commit message: 31/05/2024 Update
Other:
- note added: "ALTERNADOR"
- note removed: "GENERADOR"
Changed lines of the file:
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@@
     (effects (font (size 2.54 2.54)) (justify left bottom))
   )
-  (text "GENERADOR" (at 40.005 43.815 0)
+  (text "ALTERNADOR" (at 40.005 43.815 0)
     (effects (font (size 2.54 2.54)) (justify left bottom))
   )
