File: source/electric/ley-ohm/electric-ley-ohm-inicio-02.kicad_sch (KiCad schematic)
At the start: 59 parts

Commit message: 16/01/2025 Update
Parts:
- removed I: (no value), symbol electric-ley-ohm-inicio-rescue:current-simbolos
- removed L?: (no value), symbol electric-ley-ohm-inicio-rescue:Ley_Ohm-simbolos
- removed R: (no value), symbol electric-ley-ohm-inicio-rescue:resistencia-simbolos
- removed V: (no value), symbol electric-ley-ohm-inicio-rescue:Pila-simbolos
- added L1: Ley_Ohm, symbol electric-ley-ohm-inicio-rescue:Ley_Ohm-simbolos
- CP?: value (none) -> CopyRight
- I: value (none) -> current
- I: value (none) -> 6mA
- I: value (none) -> 0.4mA
- I: value (none) -> 8mA
- I: value (none) -> 0.25mA
- I: value (none) -> 0.2mA
- I: value (none) -> 0.05mA
- I: value (none) -> 2mA
- I: value (none) -> 0.3mA
- I: value (none) -> 3mA
- R: value (none) -> 50kΩ
- R: value (none) -> 15kΩ
- R: value (none) -> 4kΩ
- R: value (none) -> 2Ω
- R: value (none) -> 15Ω
- R: value (none) -> 6kΩ
- R: value (none) -> 10kΩ
- R: value (none) -> 80kΩ
- R: value (none) -> 5kΩ
- R: value (none) -> 120kΩ
- R: value (none) -> 60kΩ
- V: value (none) -> 6V
- V: value (none) -> 18V
- V: value (none) -> 180mV
- V: value (none) -> 24mV
- V: value (none) -> 12V
- V: value (none) -> 15V
- V: value (none) -> 9V
- V: value (none) -> 24V
Connections:
- new net: R., V. (x18)
Other:
- note added: "1kΩ = 1000Ω"
- note added: "1mA = 0.001A"
- note added: "1mV = 0.001V"
- moved on the sheet: I, R, V
