File: source/electric/ley-ohm/electric-ley-ohm-inicio.kicad_sch (KiCad schematic)
At the start: 59 parts

Commit message: 16/01/2025 Update
Parts:
- CP?: value (none) -> CopyRight
- I: value (none) -> current
- I: value (none) -> 0.1A
- I: value (none) -> 3A
- I: value (none) -> 0.5A
- I: value (none) -> 0.03A
- I: value (none) -> 2A
- I: value (none) -> 4A
- I: value (none) -> 0.2A
- I: value (none) -> 0.05A
- L?: value (none) -> Ley_Ohm
- R: value (none) -> resistencia
- R: value (none) -> 2Ω
- R: value (none) -> 120Ω
- R: value (none) -> 9Ω
- R: value (none) -> 30Ω
- R: value (none) -> 10Ω
- R: value (none) -> 100Ω
- R: value (none) -> 8Ω
- R: value (none) -> 15Ω
- R: value (none) -> 60Ω
- V: value (none) -> Pila
- V: value (none) -> 6V
- V: value (none) -> 12V
- V: value (none) -> 18V
- V: value (none) -> 9V
- V: value (none) -> 15V
- V: value (none) -> 24V
Connections:
- new net: R., V. (x19)
Other:
- moved on the sheet: I, R, V
