File: source/electric/electric-cableado/electric-cableado-3.kicad_sch (KiCad schematic)
At the start: 115 parts, among them Q1 NPN

Commit message: 22/01/2025 Update
Parts:
- removed C1: 2200uF, symbol electric-cableado-rescue:condensador_pol-simbolos
- removed C1: condensador_pol, symbol electric-cableado-rescue:condensador_pol-simbolos
- removed D1 (x10), D2 (x2): diodo_led, symbol electric-cableado-rescue:diodo_led-simbolos
- removed N?: 11, symbol electric-cableado-rescue:numero-simbolos
- removed N?: 14, symbol electric-cableado-rescue:numero-simbolos
- removed N?: 12, symbol electric-cableado-rescue:numero-simbolos
- removed N?: 13, symbol electric-cableado-rescue:numero-simbolos
- removed N?: 15, symbol electric-cableado-rescue:numero-simbolos
- removed Q1 (x2): NPN, symbol electric-cableado-rescue:NPN-simbolos
- removed Q1 (x2): NPN, symbol simbolos-electricos:NPN
- removed R1 (x3), R2 (x3), R3: resistencia, symbol electric-cableado-rescue:resistencia-simbolos
- removed R1 (x2): 10K, symbol electric-cableado-rescue:potenciometro-simbolos
- removed R1 (x2): LDR, symbol electric-cableado-rescue:LDR-simbolos
- removed R1 (x3), R2 (x2), R3: 220, symbol electric-cableado-rescue:resistencia-simbolos
- removed R2: 2K, symbol electric-cableado-rescue:resistencia-simbolos
- removed S1 (x2): switch, symbol electric-cableado-rescue:switch-simbolos
- removed S1 (x4): selector, symbol electric-cableado-rescue:selector-simbolos
- removed V1 (x5): Pila, symbol electric-cableado-rescue:Pila-simbolos
- removed V1 (x5): 5V, symbol electric-cableado-rescue:Pila-simbolos
- removed o? (x5): 1, symbol electric-cableado-rescue:conector-simbolos
- removed o? (x5): 2, symbol electric-cableado-rescue:conector-simbolos
- removed o? (x5): 3, symbol electric-cableado-rescue:conector-simbolos
- removed o? (x5): 4, symbol electric-cableado-rescue:conector-simbolos
- removed o? (x5): 5, symbol electric-cableado-rescue:conector-simbolos
- removed o? (x5): 6, symbol electric-cableado-rescue:conector-simbolos
- removed o? (x5): 7, symbol electric-cableado-rescue:conector-simbolos
- removed o? (x5): 8, symbol electric-cableado-rescue:conector-simbolos
- removed o? (x4): 9, symbol electric-cableado-rescue:conector-simbolos
- removed o? (x4): 10, symbol electric-cableado-rescue:conector-simbolos
- removed o? (x4): 11, symbol electric-cableado-rescue:conector-simbolos
- removed o? (x3): 12, symbol electric-cableado-rescue:conector-simbolos
- removed o? (x2): 13, symbol electric-cableado-rescue:conector-simbolos
- added C1: 2200uF, symbol electric-cableado-rescue:condensador_pol-simbolos
- added C1: condensador_pol, symbol electric-cableado-rescue:condensador_pol-simbolos
- added D1 (x8), D2 (x2): diodo_led, symbol electric-cableado-rescue:diodo_led-simbolos
- added M1 (x2): motor, symbol simbolos-electricos:motor
- added N10: 13, symbol electric-cableado-rescue:numero-simbolos
- added N11: 14, symbol electric-cableado-rescue:numero-simbolos
- added N12: 15, symbol electric-cableado-rescue:numero-simbolos
- added N6: 11, symbol electric-cableado-rescue:numero-simbolos
- added N9: 12, symbol electric-cableado-rescue:numero-simbolos
- added Q1: NPN, symbol electric-cableado-rescue:NPN-simbolos
- added Q1: NPN, symbol simbolos-electricos:NPN
- added R1 (x3), R2 (x2): resistencia, symbol electric-cableado-rescue:resistencia-simbolos
- added R1 (x3), R2 (x2): 220, symbol electric-cableado-rescue:resistencia-simbolos
- added R1 (x2): 10K, symbol electric-cableado-rescue:potenciometro-simbolos
- added S1 (x2): switch, symbol electric-cableado-rescue:switch-simbolos
- added S1 (x4), S2: selector, symbol electric-cableado-rescue:selector-simbolos
- added S1 (x2): interruptor, symbol simbolos-electricos:interruptor
- added S2: selector, symbol simbolos-electricos:selector
- added V1 (x5), V2: Pila, symbol electric-cableado-rescue:Pila-simbolos
- added V1 (x5), V2: 5V, symbol electric-cableado-rescue:Pila-simbolos
- added o1, o134, o139, o146, o65: 9, symbol electric-cableado-rescue:conector-simbolos
- added o106, o110, o115, o121, o59: 1, symbol electric-cableado-rescue:conector-simbolos
- added o107, o111, o116, o122, o60: 2, symbol electric-cableado-rescue:conector-simbolos
- added o108, o112, o117, o123, o61: 3, symbol electric-cableado-rescue:conector-simbolos
- added o109, o113, o118, o124, o62: 4, symbol electric-cableado-rescue:conector-simbolos
- added o114, o119, o125, o127, o63: 5, symbol electric-cableado-rescue:conector-simbolos
- added o120, o126, o128, o131, o64: 6, symbol electric-cableado-rescue:conector-simbolos
- added o129, o132, o137, o144: 7, symbol electric-cableado-rescue:conector-simbolos
- added o130, o133, o138, o145: 8, symbol electric-cableado-rescue:conector-simbolos
- added o135, o140, o147, o2, o66: 10, symbol electric-cableado-rescue:conector-simbolos
- added o136, o141, o148, o67: 11, symbol electric-cableado-rescue:conector-simbolos
- added o142, o149: 12, symbol electric-cableado-rescue:conector-simbolos
- added o143: 13, symbol electric-cableado-rescue:conector-simbolos
Connections:
- new net: D1., R1. (x3)
- new net: D1., V1.
- new net: S1., o139.
- new net: S1., o113.
- new net: R1., o133.
- new net: R1., o134.
- new net: D2., R2.
- new net: D1., D2., V1.
- new net: D1., o124.
- new net: D1., o123.
- new net: S2., o66.
- new net: D1., o118.
- new net: D1., o117.
- new net: C1., o135.
- new net: V1., o107.
- new net: V1., o106.
- new net: R2., o126.
- new net: S1., o138.
- new net: S2., V2.
- new net: S2., V1.
- new net: M1., S2.
- new net: R1., S1. (x3)
- new net: V1., o60.
- new net: D2., o120.
- new net: D1., R2.
- new net: R1., R2., V1.
- new net: V2., o61.
- new net: R2., o142.
- new net: R2., o143.
- new net: Q1., o146.
- new net: R1., o149.
- new net: R2., S1.
- new net: D1., o131.
- new net: D1., o132.
- new net: R1., o129.
- new net: R1., o130.
- new net: S1., o1.
- new net: R2., o125.
- new net: S2., o65.
- new net: C1., D1., V1.
- new net: C1., S1.
- new net: M1., o63.
- new net: V1., o116.
- new net: V1., o115.
- new net: M1., o64.
- new net: D1., o108.
- new net: S1., o127.
- new net: S1., o128.
- new net: S1., V1. (x3)
- new net: S1., V1., V2.
- new net: S1., o114.
- new net: S1., o112.
- new net: V1., o111.
- new net: S1., o2.
- new net: D1., Q1.
- new net: R1., o147.
- new net: R1., o148.
- new net: S2., o67.
- new net: V1., o122.
- new net: V1., o121.
- new net: V1., o110.
- new net: V1., o59.
- new net: D1., o109.
- new net: Q1., R1.
- new net: Q1., R1., V1.
- new net: V2., o62.
- new net: Q1., o144.
- new net: Q1., o145.
- new net: D2., o119.
- new net: R1., o141.
- new net: S1., o137.
- new net: M1., S1.
- new net: C1., o136.
- new net: R1., o140.

Commit message: 22/01/2025 Update
Connections:
- net at D1.: now also V1.; no longer R1.
- net at V1.: now also S1.; no longer D1.
- net at D2.: now also D1., V1.; no longer R2.
- net at S2.: now also M1.; no longer V2.
- net at V1.: now also S1., V2.; no longer S2.
- net at M1.: now also S1.; no longer S2.
- net at R2.: now also R1., V1.; no longer D1.
- net at R1., V1.: now also Q1.; no longer R2.
- new net: D1., R1.
- new net: D2., R2.
- new net: S2., V2.
- new net: S2., V1.
- new net: D1., R2.
- new net: C1., D1., V1.
- new net: Q1., R1.
Changed lines of the file:
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@@
 	)
 	(symbol
-		(lib_name "electric-cableado-rescue:diodo_led-simbolos")
 		(lib_id "electric-cableado-rescue:diodo_led-simbolos")
 		(at 46.355 100.33 0)
@@
 	)
 	(symbol
-		(lib_name "electric-cableado-rescue:resistencia-simbolos")
 		(lib_id "electric-cableado-rescue:resistencia-simbolos")
 		(at 193.04 149.86 270)
@@
 	)
 	(symbol
-		(lib_name "electric-cableado-rescue:diodo_led-simbolos")
 		(lib_id "electric-cableado-rescue:diodo_led-simbolos")
 		(at 64.135 213.36 0)
@@
 	)
 	(symbol
-		(lib_name "electric-cableado-rescue:diodo_led-simbolos")
 		(lib_id "electric-cableado-rescue:diodo_led-simbolos")
 		(at 114.935 257.81 0)
@@
 	)
 	(symbol
-		(lib_name "electric-cableado-rescue:diodo_led-simbolos")
 		(lib_id "electric-cableado-rescue:diodo_led-simbolos")
 		(at 114.3 204.47 0)
@@
 	)
 	(symbol
-		(lib_name "electric-cableado-rescue:Pila-simbolos")
 		(lib_id "electric-cableado-rescue:Pila-simbolos")
 		(at 115.57 81.28 0)
@@
 	)
 	(symbol
-		(lib_name "electric-cableado-rescue:resistencia-simbolos")
 		(lib_id "electric-cableado-rescue:resistencia-simbolos")
 		(at 46.355 201.93 0)
@@
 	)
 	(symbol
-		(lib_name "electric-cableado-rescue:resistencia-simbolos")
 		(lib_id "electric-cableado-rescue:resistencia-simbolos")
 		(at 57.15 271.78 0)
@@
 	)
 	(symbol
-		(lib_name "electric-cableado-rescue:resistencia-simbolos")
 		(lib_id "electric-cableado-rescue:resistencia-simbolos")
 		(at 193.04 222.25 270)
@@
 	)
 	(symbol
-		(lib_name "electric-cableado-rescue:resistencia-simbolos")
 		(lib_id "electric-cableado-rescue:resistencia-simbolos")
 		(at 64.135 201.93 0)
@@
 	)
 	(symbol
-		(lib_name "electric-cableado-rescue:resistencia-simbolos")
 		(lib_id "electric-cableado-rescue:resistencia-simbolos")
 		(at 46.355 87.63 0)
@@
 	)
 	(symbol
-		(lib_name "electric-cableado-rescue:diodo_led-simbolos")
 		(lib_id "electric-cableado-rescue:diodo_led-simbolos")
 		(at 193.04 134.62 0)
@@
 	)
 	(symbol
-		(lib_name "electric-cableado-rescue:resistencia-simbolos")
 		(lib_id "electric-cableado-rescue:resistencia-simbolos")
 		(at 193.04 96.52 270)
@@
 	)
 	(symbol
-		(lib_name "electric-cableado-rescue:condensador_pol-simbolos")
 		(lib_id "electric-cableado-rescue:condensador_pol-simbolos")
 		(at 63.5 153.67 0)
@@
 	)
 	(symbol
-		(lib_name "electric-cableado-rescue:Pila-simbolos")
 		(lib_id "electric-cableado-rescue:Pila-simbolos")
 		(at 116.84 187.96 0)
@@
 	)
 	(symbol
-		(lib_name "electric-cableado-rescue:switch-simbolos")
 		(lib_id "electric-cableado-rescue:switch-simbolos")
 		(at 182.88 82.55 0)
@@
 	)
 	(symbol
-		(lib_name "electric-cableado-rescue:switch-simbolos")
 		(lib_id "electric-cableado-rescue:switch-simbolos")
 		(at 23.495 85.09 0)
@@
 	)
 	(symbol
-		(lib_name "electric-cableado-rescue:selector-simbolos")
 		(lib_id "electric-cableado-rescue:selector-simbolos")
 		(at 124.46 163.83 0)
@@
 	)
 	(symbol
-		(lib_name "electric-cableado-rescue:Pila-simbolos")
 		(lib_id "electric-cableado-rescue:Pila-simbolos")
 		(at 15.24 149.86 0)
@@
 	)
 	(symbol
-		(lib_name "electric-cableado-rescue:diodo_led-simbolos")
 		(lib_id "electric-cableado-rescue:diodo_led-simbolos")
 		(at 57.15 262.255 0)
@@
 	)
 	(symbol
-		(lib_name "electric-cableado-rescue:potenciometro-simbolos")
 		(lib_id "electric-cableado-rescue:potenciometro-simbolos")
 		(at 190.5 269.24 0)
@@
 	)
 	(symbol
-		(lib_name "electric-cableado-rescue:Pila-simbolos")
 		(lib_id "electric-cableado-rescue:Pila-simbolos")
 		(at 116.205 241.3 0)
@@
 	)
 	(symbol
-		(lib_name "electric-cableado-rescue:Pila-simbolos")
 		(lib_id "electric-cableado-rescue:Pila-simbolos")
 		(at 115.57 134.62 0)
@@
 	)
 	(symbol
-		(lib_name "electric-cableado-rescue:resistencia-simbolos")
 		(lib_id "electric-cableado-rescue:resistencia-simbolos")
 		(at 125.095 275.59 270)
@@
 	)
 	(symbol
-		(lib_name "electric-cableado-rescue:Pila-simbolos")
 		(lib_id "electric-cableado-rescue:Pila-simbolos")
 		(at 15.875 207.01 0)
@@
 	)
 	(symbol
-		(lib_name "electric-cableado-rescue:diodo_led-simbolos")
 		(lib_id "electric-cableado-rescue:diodo_led-simbolos")
 		(at 35.56 160.02 0)
@@
 	)
 	(symbol
-		(lib_name "electric-cableado-rescue:potenciometro-simbolos")
 		(lib_id "electric-cableado-rescue:potenciometro-simbolos")
 		(at 38.1 250.19 0)
@@
 	)
 	(symbol
-		(lib_name "electric-cableado-rescue:NPN-simbolos")
 		(lib_id "electric-cableado-rescue:NPN-simbolos")
 		(at 188.595 243.84 0)
@@
 	)
 	(symbol
-		(lib_name "electric-cableado-rescue:diodo_led-simbolos")
 		(lib_id "electric-cableado-rescue:diodo_led-simbolos")
 		(at 114.3 220.98 0)
@@
 	)
 	(symbol
-		(lib_name "electric-cableado-rescue:Pila-simbolos")
 		(lib_id "electric-cableado-rescue:Pila-simbolos")
 		(at 15.875 95.25 0)
@@
 	)
 	(symbol
-		(lib_name "electric-cableado-rescue:selector-simbolos")
 		(lib_id "electric-cableado-rescue:selector-simbolos")
 		(at 55.88 142.24 180)
@@
 	)
 	(symbol
-		(lib_name "electric-cableado-rescue:selector-simbolos")
 		(lib_id "electric-cableado-rescue:selector-simbolos")
 		(at 182.88 194.31 0)
@@
 	)
 	(symbol
-		(lib_name "simbolos-electricos:NPN")
 		(lib_id "simbolos-electricos:NPN")
 		(at 50.8 250.19 0)
@@
 	)
 	(symbol
-		(lib_name "electric-cableado-rescue:resistencia-simbolos")
 		(lib_id "electric-cableado-rescue:resistencia-simbolos")
 		(at 35.56 148.59 0)
@@
 	)
 	(symbol
-		(lib_name "electric-cableado-rescue:resistencia-simbolos")
 		(lib_id "electric-cableado-rescue:resistencia-simbolos")
 		(at 193.04 208.28 270)
@@
 	)
 	(symbol
-		(lib_name "electric-cableado-rescue:condensador_pol-simbolos")
 		(lib_id "electric-cableado-rescue:condensador_pol-simbolos")
 		(at 193.04 165.1 0)
@@
 	)
 	(symbol
-		(lib_name "electric-cableado-rescue:diodo_led-simbolos")
 		(lib_id "electric-cableado-rescue:diodo_led-simbolos")
 		(at 46.355 213.36 0)
@@
 	)
 	(symbol
-		(lib_name "electric-cableado-rescue:selector-simbolos")
 		(lib_id "electric-cableado-rescue:selector-simbolos")
 		(at 24.765 195.58 0)
@@
 	)
 	(symbol
-		(lib_name "electric-cableado-rescue:diodo_led-simbolos")
 		(lib_id "electric-cableado-rescue:diodo_led-simbolos")
 		(at 114.3 97.79 0)
@@
 	)
 	(symbol
-		(lib_name "electric-cableado-rescue:Pila-simbolos")
 		(lib_id "electric-cableado-rescue:Pila-simbolos")
 		(at 15.875 259.08 0)

Commit message: 25/01/2025 Update
Parts:
- o1: value 9 -> 7
- o2: value 10 -> 8
Connections:
- net at D1.: now also V1.; no longer R1.
- net at V1.: now also S1.; no longer D1.
- net at D2.: now also D1., V1.; no longer R2.
- net at S2.: now also M1.; no longer V2.
- net at V1.: now also S1., V2.; no longer S2.
- net at M1.: now also S1.; no longer S2.
- net at R2.: now also R1., V1.; no longer D1.
- net at R1., V1.: now also Q1.; no longer R2.
- new net: D1., R1.
- new net: D2., R2.
- new net: S2., V2.
- new net: S2., V1.
- new net: D1., R2.
- new net: C1., D1., V1.
- new net: Q1., R1.
Other:
- moved on the sheet: D1, D2, Q1, R1, R2, S1, S2, V1
