File: source/electric/electric-cableado/electric-cableado-2.kicad_sch (KiCad schematic)
At the start: 111 parts

Commit message: 22/01/2025 Update
Connections:
- net at V1.: now also S2.; no longer S1.
- net at S2.: now also L1.; no longer V1.
- net at L2.: now also S2.; no longer S1.
- net at S1., S2.: no longer L1.
- net at S1.: now also L1., S2.; no longer V1.
- net at S1.: now also L2., S2.; no longer V1.
- net at L2., S2.: now also L1.; no longer S1.
- new net: L1., L2., V1. (x2)
- new net: S1., V1. (x3)
- new net: L2., S1.
- new net: L1., S1., S2.

Commit message: 25/01/2025 Update
Connections:
- net at V1.: now also S2.; no longer S1.
- net at S2.: now also L1.; no longer V1.
- net at L2.: now also S2.; no longer S1.
- net at S1., S2.: no longer L1.
- net at S1.: now also L1., S2.; no longer V1.
- net at S1.: now also L2., S2.; no longer V1.
- net at L2., S2.: now also L1.; no longer S1.
- new net: L1., L2., V1. (x2)
- new net: S1., V1. (x3)
- new net: L2., S1.
- new net: L1., S1., S2.
Other:
- moved on the sheet: L1, L2, S1, S2, V1

Commit message: 25/01/2025 Update
Parts:
- renumbered L2 to L1, L1 to L2
Connections:
- net at V1.: now also S2.; no longer S1.
- net at S2.: now also L1.; no longer V1.
- net at L2.: now also S2.; no longer S1.
- net at S1., S2.: no longer L1.
- net at S1.: now also L1., S2.; no longer V1. (x2)
- net at L1., S2.: now also L2.; no longer S1.
- new net: L1., L2., V1. (x2)
- new net: S1., V1. (x3)
- new net: L2., S1.
- new net: L1., S1., S2.
Changed lines of the file:
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@@
 	)
 	(symbol
+		(lib_name "electric-cableado-rescue:lampara-simbolos")
 		(lib_id "electric-cableado-rescue:lampara-simbolos")
 		(at 44.45 104.14 0)
@@
 		(on_board yes)
 		(dnp no)
-		(property "Reference" "L1"
+		(property "Reference" "L2"
 			(at 48.26 109.22 0)
 			(effects
@@
 			(project "electric-cableado"
 				(path "/ed402a02-18b5-4b69-8c2e-4a17e0d73589/00000000-0000-0000-0000-000061659b7a"
-					(reference "L1")
+					(reference "L2")
 					(unit 1)
 				)
@@
 	)
 	(symbol
+		(lib_name "electric-cableado-rescue:lampara-simbolos")
 		(lib_id "electric-cableado-rescue:lampara-simbolos")
 		(at 44.45 88.9 0)
@@
 		(on_board yes)
 		(dnp no)
-		(property "Reference" "L2"
+		(property "Reference" "L1"
 			(at 48.26 93.98 0)
 			(effects
@@
 			(project "electric-cableado"
 				(path "/ed402a02-18b5-4b69-8c2e-4a17e0d73589/00000000-0000-0000-0000-000061659b7a"
-					(reference "L2")
-					(unit 1)
-				)
+					(reference "L1")
+					(unit 1)
+				)

Commit message: 26/01/2025 Update
Connections:
- net at V1.: now also S2.; no longer S1.
- net at S2.: now also L1.; no longer V1.
- net at L2.: now also S2.; no longer S1.
- net at S1., S2.: no longer L1.
- net at S1.: now also L1., S2.; no longer V1. (x2)
- net at L1., S2.: now also L2.; no longer S1.
- new net: L1., L2., V1. (x2)
- new net: S1., V1. (x3)
- new net: L2., S1.
- new net: L1., S1., S2.
Changed lines of the file:
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@@
 	)
 	(symbol
-		(lib_name "electric-cableado-rescue:lampara-simbolos")
 		(lib_id "electric-cableado-rescue:lampara-simbolos")
 		(at 44.45 104.14 0)
@@
 	)
 	(symbol
-		(lib_name "electric-cableado-rescue:lampara-simbolos")
 		(lib_id "electric-cableado-rescue:lampara-simbolos")
 		(at 44.45 88.9 0)
