File: source/electric/electric-cableado/electric-cableado-4.kicad_sch (KiCad schematic)
At the start: 132 parts, among them Q1 NPN, Q2 NPN, U1 L7805, U2 L7805

Commit message: 22/01/2025 Update
Parts:
- renumbered U2 to U1
Connections:
- net at R3.: now also Q1.; no longer D1.
- net at Q1.: now also R2., V1.; no longer R3.
- net at R1., TR1.: no longer V1.
- new net: D1., R3.
- new net: Q1., R1., R2.
- new net: C1., C2., C3., U1.2 (GND), V1., o35.
- new net: C1., L1., Q1., Q2., V1.
- new net: D1., Q1., V1.
- new net: D1., Q1., TR1.
- new net: D2., R1., V1.
- new net: D1., Q1., R1.
- new net: R1., TR1., V1.
Changed lines of the file:
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@@
 	)
 	(symbol
-		(lib_name "electric-cableado-rescue:resistencia-simbolos")
 		(lib_id "electric-cableado-rescue:resistencia-simbolos")
 		(at 59.055 95.25 0)
@@
 	)
 	(symbol
-		(lib_name "electric-cableado-rescue:LDR-simbolos")
 		(lib_id "electric-cableado-rescue:LDR-simbolos")
 		(at 33.655 85.09 0)
@@
 	)
 	(symbol
-		(lib_name "electric-cableado-rescue:resistencia-simbolos")
 		(lib_id "electric-cableado-rescue:resistencia-simbolos")
 		(at 193.675 115.57 270)
@@
 	)
 	(symbol
-		(lib_name "electric-cableado-rescue:NPN-simbolos")
 		(lib_id "electric-cableado-rescue:NPN-simbolos")
 		(at 188.595 82.55 0)
@@
 	)
 	(symbol
-		(lib_name "electric-cableado-rescue:LDR-simbolos")
 		(lib_id "electric-cableado-rescue:LDR-simbolos")
 		(at 125.095 115.57 270)
@@
 	)
 	(symbol
-		(lib_name "electric-cableado-rescue:Pila-simbolos")
 		(lib_id "electric-cableado-rescue:Pila-simbolos")
 		(at 116.205 81.28 0)
@@
 	)
 	(symbol
-		(lib_name "electric-cableado-rescue:resistencia-simbolos")
 		(lib_id "electric-cableado-rescue:resistencia-simbolos")
 		(at 33.655 107.95 0)
@@
 	)
 	(symbol
-		(lib_name "electric-cableado-rescue:Pila-simbolos")
 		(lib_id "electric-cableado-rescue:Pila-simbolos")
 		(at 15.875 97.79 0)
@@
 	)
 	(symbol
-		(lib_name "electric-cableado-rescue:diodo_led-simbolos")
 		(lib_id "electric-cableado-rescue:diodo_led-simbolos")
 		(at 59.055 85.09 0)
@@
 	)
 	(symbol
-		(lib_name "electric-cableado-rescue:diodo_led-simbolos")
 		(lib_id "electric-cableado-rescue:diodo_led-simbolos")
 		(at 114.935 97.79 0)
@@
 	)
 	(symbol
-		(lib_name "simbolos-electricos:condensador")
 		(lib_id "simbolos-electricos:condensador")
 		(at 79.375 156.21 0)
@@
 	)
 	(symbol
-		(lib_name "simbolos-electricos:inductancia")
 		(lib_id "simbolos-electricos:inductancia")
 		(at 37.465 243.84 0)
@@
 	)
 	(symbol
-		(lib_name "electric-cableado-rescue:diodo_led-simbolos")
 		(lib_id "electric-cableado-rescue:diodo_led-simbolos")
 		(at 183.515 24.13 90)
@@
 	)
 	(symbol
-		(lib_name "electric-cableado-rescue:Pila-simbolos")
 		(lib_id "electric-cableado-rescue:Pila-simbolos")
 		(at 15.875 156.21 0)
@@
 	)
 	(symbol
-		(lib_name "electric-cableado-rescue:Pila-simbolos")
 		(lib_id "electric-cableado-rescue:Pila-simbolos")
 		(at 116.205 134.62 0)
@@
 	)
 	(symbol
-		(lib_name "electric-cableado-rescue:NPN-simbolos")
 		(lib_id "electric-cableado-rescue:NPN-simbolos")
 		(at 119.38 258.445 0)
@@
 	)
 	(symbol
-		(lib_name "electric-cableado-rescue:NPN-simbolos")
 		(lib_id "electric-cableado-rescue:NPN-simbolos")
 		(at 188.595 189.23 0)
@@
 	)
 	(symbol
-		(lib_name "simbolos-electricos:NPN")
 		(lib_id "simbolos-electricos:NPN")
 		(at 39.37 214.63 0)
@@
 	)
 	(symbol
-		(lib_name "electric-cableado-rescue:resistencia-simbolos")
 		(lib_id "electric-cableado-rescue:resistencia-simbolos")
 		(at 34.29 29.21 0)
@@
 	)
 	(symbol
-		(lib_name "electric-cableado-rescue:resistencia-simbolos")
 		(lib_id "electric-cableado-rescue:resistencia-simbolos")
 		(at 193.04 60.325 270)
@@
 	)
 	(symbol
-		(lib_name "electric-cableado-rescue:Pila-simbolos")
 		(lib_id "electric-cableado-rescue:Pila-simbolos")
 		(at 15.875 261.62 0)
@@
 	)
 	(symbol
-		(lib_name "simbolos-electricos:transformador")
 		(lib_id "simbolos-electricos:transformador")
 		(at 116.84 204.47 0)
@@
 	)
 	(symbol
-		(lib_name "simbolos-electricos:NPN")
 		(lib_id "simbolos-electricos:NPN")
 		(at 31.115 257.81 0)
@@
 	)
 	(symbol
-		(lib_name "electric-cableado-rescue:diodo_led-simbolos")
 		(lib_id "electric-cableado-rescue:diodo_led-simbolos")
 		(at 53.34 29.21 0)
@@
 	)
 	(symbol
-		(lib_name "electric-cableado-rescue:resistencia-simbolos")
 		(lib_id "electric-cableado-rescue:resistencia-simbolos")
 		(at 37.465 270.51 0)
@@
 	)
 	(symbol
-		(lib_name "electric-cableado-rescue:Pila-simbolos")
 		(lib_id "electric-cableado-rescue:Pila-simbolos")
 		(at 116.84 241.3 0)
@@
 	)
 	(symbol
-		(lib_name "electric-cableado-rescue:Pila-simbolos")
 		(lib_id "electric-cableado-rescue:Pila-simbolos")
 		(at 15.24 41.91 0)
@@
 	)
 	(symbol
-		(lib_name "electric-cableado-rescue:Pila-simbolos")
 		(lib_id "electric-cableado-rescue:Pila-simbolos")
 		(at 15.875 204.47 0)
@@
 	)
 	(symbol
-		(lib_name "simbolos-electricos:condensador")
 		(lib_id "simbolos-electricos:condensador")
 		(at 193.675 168.91 270)
@@
 	)
 	(symbol
-		(lib_name "simbolos-electricos:condensador")
 		(lib_id "simbolos-electricos:condensador")
 		(at 114.935 171.45 90)
@@
 	)
 	(symbol
-		(lib_name "electric-cableado-rescue:resistencia-simbolos")
 		(lib_id "electric-cableado-rescue:resistencia-simbolos")
 		(at 193.675 222.25 270)
@@
 	)
 	(symbol
-		(lib_name "simbolos-electricos:inductancia")
 		(lib_id "simbolos-electricos:inductancia")
 		(at 193.04 240.03 270)
@@
 	)
 	(symbol
-		(lib_name "simbolos-electricos:condensador")
 		(lib_id "simbolos-electricos:condensador")
 		(at 33.02 156.21 0)
@@
 	)
 	(symbol
-		(lib_name "electric-cableado-rescue:resistencia-simbolos")
 		(lib_id "electric-cableado-rescue:resistencia-simbolos")
 		(at 114.3 43.18 90)
@@
 	)
 	(symbol
-		(lib_name "simbolos-electricos:NPN")
 		(lib_id "simbolos-electricos:NPN")
 		(at 52.705 107.95 0)
@@
 	)
 	(symbol
-		(lib_name "electric-cableado-rescue:Pila-simbolos")
 		(lib_id "electric-cableado-rescue:Pila-simbolos")
 		(at 115.57 25.4 0)
@@
 	)
 	(symbol
-		(lib_name "electric-cableado-rescue:diodo_led-simbolos")
 		(lib_id "electric-cableado-rescue:diodo_led-simbolos")
 		(at 184.785 208.28 90)
@@
 	)
 	(symbol
-		(lib_name "simbolos-electricos:condensador")
 		(lib_id "simbolos-electricos:condensador")
 		(at 191.77 255.27 270)
@@
 	)
 	(symbol
-		(lib_name "electric-cableado-rescue:NPN-simbolos")
 		(lib_id "electric-cableado-rescue:NPN-simbolos")
 		(at 187.96 40.64 0)
@@
 	)
 	(symbol
-		(lib_name "simbolos-electricos:condensador")
 		(lib_id "simbolos-electricos:condensador")
 		(at 51.435 244.475 0)
@@
 	)
 	(symbol
-		(lib_name "electric-cableado-rescue:resistencia-simbolos")
 		(lib_id "electric-cableado-rescue:resistencia-simbolos")
 		(at 53.34 53.975 0)
@@
 	)
 	(symbol
-		(lib_name "simbolos-electricos:diodo_zener")
 		(lib_id "simbolos-electricos:diodo_zener")
 		(at 34.29 61.595 180)
@@
 	)
 	(symbol
-		(lib_name "electric-cableado-rescue:resistencia-simbolos")
 		(lib_id "electric-cableado-rescue:resistencia-simbolos")
 		(at 193.675 101.6 270)
@@
 	)
 	(symbol
-		(lib_name "electric-cableado-rescue:Pila-simbolos")
 		(lib_id "electric-cableado-rescue:Pila-simbolos")
 		(at 116.205 187.96 0)
@@
 	)
 	(symbol
-		(lib_name "simbolos-electricos:diodo_zener")
 		(lib_id "simbolos-electricos:diodo_zener")
 		(at 116.205 59.69 90)
@@
 		(on_board yes)
 		(dnp no)
-		(property "Reference" "U2"
+		(property "Reference" "U1"
 			(at 117.729 147.193 0)
 			(effects
@@
 			(project "electric-cableado"
 				(path "/ed402a02-18b5-4b69-8c2e-4a17e0d73589/202af1f8-3938-4e13-90b7-bd419a08a5d7"
-					(reference "U2")
+					(reference "U1")
 					(unit 1)
 				)
@@
 	)
 	(symbol
-		(lib_name "simbolos-electricos:NPN")
 		(lib_id "simbolos-electricos:NPN")
 		(at 59.055 257.81 0)
@@
 	)
 	(symbol
-		(lib_name "electric-cableado-rescue:diodo_led-simbolos")
 		(lib_id "electric-cableado-rescue:diodo_led-simbolos")
 		(at 60.96 215.9 0)
@@
 	)
 	(symbol
-		(lib_name "simbolos-electricos:NPN")
 		(lib_id "simbolos-electricos:NPN")
 		(at 46.99 41.91 0)
@@
 	)
 	(symbol
-		(lib_name "simbolos-electricos:condensador")
 		(lib_id "simbolos-electricos:condensador")
 		(at 61.595 156.21 0)
@@
 	)
 	(symbol
-		(lib_name "electric-cableado-rescue:resistencia-simbolos")
 		(lib_id "electric-cableado-rescue:resistencia-simbolos")
 		(at 31.75 190.5 0)
@@
 	)
 	(symbol
-		(lib_name "electric-cableado-rescue:NPN-simbolos")
 		(lib_id "electric-cableado-rescue:NPN-simbolos")
 		(at 187.96 271.78 0)
@@
 	)
 	(symbol
-		(lib_name "simbolos-electricos:condensador")
 		(lib_id "simbolos-electricos:condensador")
 		(at 193.675 154.94 270)
@@
 	)
 	(symbol
-		(lib_name "electric-cableado-rescue:resistencia-simbolos")
 		(lib_id "electric-cableado-rescue:resistencia-simbolos")
 		(at 114.3 276.86 90)

Commit message: 25/01/2025 Update
Parts:
- U1: value L7805 -> 7805
- o30: value 10 -> 12
- o31: value 11 -> 13
- o37: value 8 -> 10
- o38: value 9 -> 11
Connections:
- net at R3.: now also Q1.; no longer D1.
- net at Q1.: now also R2., V1.; no longer R3.
- net at R1., TR1.: no longer V1.
- new net: D1., R3.
- new net: Q1., R1., R2.
- new net: C1., C2., C3., U1.2 (GND), V1., o35.
- new net: C1., L1., Q1., Q2., V1.
- new net: D1., Q1., V1.
- new net: D1., Q1., TR1.
- new net: D2., R1., V1.
- new net: D1., Q1., R1.
- new net: R1., TR1., V1.
Other:
- note added: "8"
- note added: "9"
- moved on the sheet: C1, C2, C3, D1, L1, Q1, Q2, R1, R2, R3, TR1, U1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

Commit message: 25/01/2025 Update
Connections:
- net at R3.: now also Q1.; no longer D1.
- net at Q1.: now also R2., V1.; no longer R3.
- net at R1., TR1.: no longer V1.
- new net: D1., R3.
- new net: Q1., R1., R2.
- new net: C1., C2., C3., U1.2 (GND), V1., o35.
- new net: C1., L1., Q1., Q2., V1.
- new net: D1., Q1., V1.
- new net: D1., Q1., TR1.
- new net: D2., R1., V1.
- new net: D1., Q1., R1.
- new net: R1., TR1., V1.
Changed lines of the file:
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@@
 	)
 	(symbol
-		(lib_name "electric-cableado-rescue:resistencia-simbolos")
 		(lib_id "electric-cableado-rescue:resistencia-simbolos")
 		(at 193.04 114.3 270)
@@
 	)
 	(symbol
-		(lib_name "electric-cableado-rescue:NPN-simbolos")
 		(lib_id "electric-cableado-rescue:NPN-simbolos")
 		(at 187.96 81.28 0)
@@
 	)
 	(symbol
-		(lib_name "electric-cableado-rescue:LDR-simbolos")
 		(lib_id "electric-cableado-rescue:LDR-simbolos")
 		(at 124.46 114.3 270)
@@
 	)
 	(symbol
-		(lib_name "electric-cableado-rescue:Pila-simbolos")
 		(lib_id "electric-cableado-rescue:Pila-simbolos")
 		(at 115.57 80.01 0)
@@
 	)
 	(symbol
-		(lib_name "electric-cableado-rescue:diodo_led-simbolos")
 		(lib_id "electric-cableado-rescue:diodo_led-simbolos")
 		(at 114.3 96.52 0)
@@
 	)
 	(symbol
-		(lib_name "electric-cableado-rescue:Pila-simbolos")
 		(lib_id "electric-cableado-rescue:Pila-simbolos")
 		(at 115.57 134.62 0)
@@
 	)
 	(symbol
-		(lib_name "electric-cableado-rescue:NPN-simbolos")
 		(lib_id "electric-cableado-rescue:NPN-simbolos")
 		(at 187.96 190.5 0)
@@
 	)
 	(symbol
-		(lib_name "simbolos-electricos:transformador")
 		(lib_id "simbolos-electricos:transformador")
 		(at 116.205 205.74 0)
@@
 	)
 	(symbol
-		(lib_name "simbolos-electricos:condensador")
 		(lib_id "simbolos-electricos:condensador")
 		(at 193.04 168.91 270)
@@
 	)
 	(symbol
-		(lib_name "simbolos-electricos:condensador")
 		(lib_id "simbolos-electricos:condensador")
 		(at 114.3 171.45 90)
@@
 	)
 	(symbol
-		(lib_name "electric-cableado-rescue:resistencia-simbolos")
 		(lib_id "electric-cableado-rescue:resistencia-simbolos")
 		(at 193.04 223.52 270)
@@
 	)
 	(symbol
-		(lib_name "electric-cableado-rescue:diodo_led-simbolos")
 		(lib_id "electric-cableado-rescue:diodo_led-simbolos")
 		(at 184.15 209.55 90)
@@
 	)
 	(symbol
-		(lib_name "electric-cableado-rescue:resistencia-simbolos")
 		(lib_id "electric-cableado-rescue:resistencia-simbolos")
 		(at 193.04 100.33 270)
@@
 	)
 	(symbol
-		(lib_name "electric-cableado-rescue:Pila-simbolos")
 		(lib_id "electric-cableado-rescue:Pila-simbolos")
 		(at 115.57 189.23 0)
@@
 	)
 	(symbol
-		(lib_name "simbolos-electricos:condensador")
 		(lib_id "simbolos-electricos:condensador")
 		(at 193.04 154.94 270)

Commit message: 26/01/2025 Update
Connections:
- net at R3.: now also Q1.; no longer D1.
- net at Q1.: now also R2., V1.; no longer R3.
- net at C2., C3., o34.: now also U1. (OUT); no longer U1.3 (OUT)
- net at o20.: now also U1. (OUT); no longer U1.3 (OUT)
- net at C1., V1.: now also U1. (OUT); no longer U1.1 (IN)
- net at o28.: now also U1. (OUT); no longer U1.1 (IN)
- net at o21.: now also U1. (OUT); no longer U1.2 (GND)
- net at R1., TR1.: no longer V1.
- new net: D1., R3.
- new net: Q1., R1., R2.
- new net: C1., C2., C3., U1. (OUT), V1., o35.
- new net: C1., L1., Q1., Q2., V1.
- new net: D1., Q1., V1.
- new net: D1., Q1., TR1.
- new net: D2., R1., V1.
- new net: D1., Q1., R1.
- new net: R1., TR1., V1.
Changed lines of the file:
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@@
 		)
 		(property "Value" "GND"
-			(at 93.472 173.99 0)
+			(at 87.884 170.942 0)
 			(effects
 				(font
@@
 		)
 		(property "Value" "V+"
-			(at 92.202 146.812 0)
+			(at 88.392 143.51 0)
 			(effects
 				(font
@@
 		)
 		(property "Value" "7805"
-			(at 120.015 158.877 0)
+			(at 116.713 163.195 90)
 			(effects
 				(font
@@
 			)
 		)
-		(pin "3"
+		(pin ""
 		)
-		(pin "2"
+		(pin ""
 		)
-		(pin "1"
+		(pin ""
 		)
 		(instances
@@
 			)
 		)
-		(pin "3"
+		(pin ""
 		)
-		(pin "2"
+		(pin ""
 		)
-		(pin "1"
+		(pin ""
 		)
 		(instances
