File: source/electric/serie-paralelo/electric-serie-paralelo.kicad_sch (KiCad schematic)
At the start: 61 parts

Commit message: 29/01/2025 Update
Parts:
- removed CP1: CopyRight, symbol electric-serie-paralelo-rescue:CopyRight-simbolos
- added CP2: CopyRight, symbol electric-serie-paralelo-rescue:CopyRight-simbolos
Connections:
- net at L1.: now also V.; no longer L5.
- net at V.: now also L5.; no longer L1.
- net at V.: now also L15.; no longer L11.
- net at L15.: now also L11.; no longer V.
- net at L18.: now also V.; no longer L22.
- net at V.: now also L22.; no longer L18.
- net at L28., V.: no longer L32.
- net at L25.: now also V.; no longer L29.
- net at V.: now also L29.; no longer L25.
- net at V.: now also L37.; no longer L34.
- net at L37.: now also L34.; no longer V.
- net at L38., V.: no longer L35.
- new net: L1., L5.
- new net: L4., L8., V.
- new net: L2., L6., V.
- new net: L12., L16., V.
- new net: L13., L9., V.
- new net: L11., V.
- new net: L17., L21., V.
- new net: L18., L22.
- new net: L19., L23., V.
- new net: L26., L30., V.
- new net: L27., L31., V.
- new net: L28., L32., V.
- new net: L25., L29.
- new net: L33., L40., V.
- new net: L34., V.
- new net: L35., L38., V.
