File: source/electronic/pcb-luces-led/electronic-pcb-luces-led.kicad_sch (KiCad schematic)
At the start: 22 parts, among them SW1 SW_SPDT, U1 74HC14

Commit message: 11/12/2025 Update
Parts:
- BT1: footprint electronic-pcb-luces-led:PinHeader_1x02_P2.54mm_Vertical -> footprints:PinHeader_1x02_P2.54mm_Vertical
- C1, C2, C3: footprint electronic-pcb-luces-led:CP_Radial_D5.0mm_P2.00mm -> footprints:CP_Radial_D5.0mm_P2.00mm
- C4: footprint electronic-pcb-luces-led:C_Rect_L9.0mm_W3.2mm_P7.50mm_MKT -> footprints:C_Rect_L9.0mm_W3.2mm_P7.50mm_MKT
- D1, D2, D3, D4, D5, D6: footprint electronic-pcb-luces-led:LED_D5.0mm -> footprints:LED_D5.0mm
- R1, R2, R4, R5, R7, R8: value 220 -> 180; footprint electronic-pcb-luces-led:R_Axial_DIN0411_L9.9mm_D3.6mm_P12.70mm_Horizontal -> footprints:R_Axial_DIN0411_L9.9mm_D3.6mm_P12.70mm_Horizontal
- R3: footprint electronic-pcb-luces-led:R_Axial_DIN0411_L9.9mm_D3.6mm_P12.70mm_Horizontal -> footprints:R_Axial_DIN0411_L9.9mm_D3.6mm_P12.70mm_Horizontal
- R6: value 220K -> 330K; footprint electronic-pcb-luces-led:R_Axial_DIN0411_L9.9mm_D3.6mm_P12.70mm_Horizontal -> footprints:R_Axial_DIN0411_L9.9mm_D3.6mm_P12.70mm_Horizontal
- R9: value 220K -> 470K; footprint electronic-pcb-luces-led:R_Axial_DIN0411_L9.9mm_D3.6mm_P12.70mm_Horizontal -> footprints:R_Axial_DIN0411_L9.9mm_D3.6mm_P12.70mm_Horizontal
- SW1: footprint electronic-pcb-luces-led:SW_Slide_1P2T_CK_OS102011MS2Q -> footprints:SW_Slide_1P2T_CK_OS102011MS2Q
- U1: footprint electronic-pcb-luces-led:DIP-14_W7.62mm_Socket_LongPads -> footprints:DIP-14_W7.62mm_Socket_LongPads
