File: source/arduprog/stroboscope/schematics/stroboscope-lamp.kicad_sch (KiCad schematic)
At the start: 45 parts, among them Q1 BC337-25, Q2 BC337-25, Q3 BC337-25, Q4 BC337-25, Q5 BC337-25

Commit message: 17/03/2026 Update
Parts:
- removed R11, R13, R5, R7, R9: 100, symbol simbolos-electronicos:resistencia
- renumbered C2 to C3, D9 to D10, D10 to D11, D11 to D12, D12 to D13, D13 to D14, D14 to D15, D15 to D16, D16 to D17, D17 to D18, D18 to D19, D1 to D2, D19 to D20, D20 to D21, D21 to D22, D22 to D23, D23 to D24, D24 to D25, D25 to D26, D26 to D27, D2 to D3, D3 to D4, D4 to D5, D5 to D6, D6 to D7, D7 to D8, D8 to D9, Q1 to Q2, Q2 to Q3, Q3 to Q4, Q4 to Q5, Q5 to Q6, R14 to R10, R4 to R5, R8 to R7, R10 to R8, R12 to R9, V9 to V8, V10 to V9
Connections:
- net at D5.: now also D4.; no longer D6.
- net at D4.: now also D3.; no longer D5.
- net at D14.: now also D15.; no longer D13.
- net at Q3.: now also D12.; no longer R7.
- net at D21.: now also D22.; no longer D20.
- net at D22.: now also Q5.; no longer D21.
- net at Q2.: now also D7.; no longer R6.
- net at D7.: now also D6.; no longer Q2.
- net at D11.: now also D10.; no longer D12.
- net at D25.: now also D26.; no longer D24.
- net at D26.: now also D27.; no longer D25.
- net at Q6.: now also R10.; no longer D27.
- net at Q4.: now also D17.; no longer R8.
- net at D10.: now also D9.; no longer D11.
- net at D9.: now also D8.; no longer D10.
- net at Q5.: now also R9.; no longer D22.
- net at D15.: now also D16.; no longer D14.
- new net: D5., D6.
- new net: D13., D14.
- new net: Q3., R7.
- new net: D20., D21.
- new net: D2., Q2., Q3., Q4., Q5., Q6., R5.
- new net: Q2., R6.
- new net: D11., D12.
- new net: D24., D25.
- new net: D27., Q6.
- new net: Q4., R8.
- new net: D16., D17.
Other:
- note added: "D2 = RED LED HIGH BRIGHTNESS (1.8V, 20mA, 5mm diameter)"
- note added: "D3 - D27 = WHITE LED (0.5W, 3.3V, 150mA, 8mm diameter)"
- note removed: "D1 = RED LED HIGH BRIGHTNESS (1.8V, 20mA, 5mm diameter)"
- note removed: "D2 - D26 = WHITE LED (0.5W, 3.3V, 150mA, 8mm diameter)"
- note removed: "R6, R8, R10, R12, R14 = 1/4W resistor"

Commit message: 22/03/2026 Update
Parts:
- removed D2: diodo_led, symbol simbolos-electronicos:diodo_led
- added Q2: BC337-25, symbol simbolos-electronicos:NPN
- R10: renamed from R9; value 3.3 -> 2.2
- R11: renamed from R10; value 3.3 -> 2.2
- R7: renamed from R6; value 3.3 -> 2.2
- R8: renamed from R7; value 3.3 -> 2.2
- R9: renamed from R8; value 3.3 -> 2.2
- renumbered D11 to D10, D12 to D11, D13 to D12, D14 to D13, D15 to D14, D16 to D15, D17 to D16, D18 to D17, D19 to D18, D20 to D19, D3 to D2, D21 to D20, D22 to D21, D23 to D22, D24 to D23, D25 to D24, D26 to D25, D27 to D26, D4 to D3, D5 to D4, D6 to D5, D7 to D6, D8 to D7, D9 to D8, D10 to D9, Q2 to Q3, Q3 to Q4, Q4 to Q5, Q5 to Q6, Q6 to Q7, R5 to R6
Connections:
- net GND: now also Q2.
- net at D4.: now also D3.; no longer D5.
- net at D3.: now also D2.; no longer D4.
- net at D13.: now also D14.; no longer D12.
- net at Q4.: now also D11.; no longer R8.
- net at D20.: now also D21.; no longer D19.
- net at D21.: now also Q6.; no longer D20.
- net at Q3.: now also D6.; no longer R7.
- net at D6.: now also D5.; no longer Q3.
- net at D10.: now also D9.; no longer D11.
- net at D24.: now also D25.; no longer D23.
- net at D25.: now also D26.; no longer D24.
- net at Q7.: now also R11.; no longer D26.
- net at Q5.: now also D16.; no longer R9.
- net at D9.: now also D8.; no longer D10.
- net at D8.: now also D7.; no longer D9.
- net at Q6.: now also R10.; no longer D21.
- net at D14.: now also D15.; no longer D13.
- net LAMP-GATE renamed LAMP-ON
- new net: D4., D5.
- new net: D12., D13.
- new net: Q4., R8.
- new net: D19., D20.
- new net: Q2., Q3., Q4., Q5., Q6., Q7., R6.
- new net: Q2., Q3., R7.
- new net: D10., D11.
- new net: D23., D24.
- new net: D26., Q7.
- new net: Q5., R9.
- new net: D15., D16.
Other:
- note added: "D2 - D26 = WHITE LED (0.5W, 3.3V, 150mA, 8mm diameter)"
- note removed: "D2 = RED LED HIGH BRIGHTNESS (1.8V, 20mA, 5mm diameter)"
- note removed: "D3 - D27 = WHITE LED (0.5W, 3.3V, 150mA, 8mm diameter)"
- note removed: "VCC (+20V)"
- moved on the sheet: R10, R11, R6, R7, R8, R9
