File: source/arduprog/stroboscope/schematics/stroboscope.kicad_sch (KiCad schematic)
At the start: 19 parts

Commit message: 17/03/2026 Update
Parts:
- removed U2: ~, symbol simbolos-electronicos:BOOST
- removed V6: tierra, symbol simbolos-electronicos:tierra
- added C1: 100nF, symbol simbolos-electronicos:condensador
- added D1: 1N5819, symbol simbolos-electronicos:diodo
- added L1: 100uH, symbol simbolos-electronicos:inductancia
- added Q1: IRLZ44N, symbol simbolos-electronicos:MOSFET_N
- added R1: 100, symbol simbolos-electronicos:resistencia
- added S5: interruptor, symbol simbolos-electronicos:interruptor
- R3: renamed from R2; value 4K7 -> 10K
- S1, S2, S3, S4: value pulsador_na -> ~
- renumbered C1 to C2, R1 to R2, R3 to R4, V8 to V1, V1 to V3, V7 to V5, V5 to V6, V3 to V7
Connections:
- net VTEST is gone; now on net BOOST_V: A1.20 (A1), R3., R4.
- net +5V: no longer R2.~
- net VBAT: now also C1., L1., S5.; no longer V4.
- net BOOST_G: now reaches A1.14 (D11)
- net BOOST_G: now also Q1.
- net +3.3V: now reaches A1.17 (3V3)
- net +3.3V: now also R2.~, R1.
- net at A1.18 (AREF): now also R1.
- net +22V: now reaches C2.
- net +22V: now also R3., D1.; no longer R4.
- net at V6.: now also C2., R4., C1., Q1.
- net +20V renamed BOOST_V
- net BOOST_V: no longer C2.
- net GATE renamed LAMP_ON
- new net: D1., L1., Q1.
- new net: R2.~, S1., S2., S3., S4., V1.
- new net: S5., V4.
- no-connect marks 17 -> 14
Other:
- note added: "LED LAMP"
- moved on the sheet: R3, R4

Commit message: 22/03/2026 Update
Parts:
- added R3: 10K, symbol simbolos-electronicos:resistencia
- renumbered R3 to R4, R4 to R5
Connections:
- net BOOST_G: now also R3.
- net +22V renamed LAMP-VCC
- new net: D1., L1., Q1.
- new net: C1., C2., Q1., R3., R5., V6.
- new net: R2.~, S1., S2., S3., S4., V1.
Other:
- sheet stroboscope-lamp ports: added LAMP-ON; removed LAMP-GATE
- moved on the sheet: C2
Changed lines of the file:
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@@
 		(title "Stroboscope LED for Arduino")
 		(date "2026-03-06")
-		(rev "R1")
+		(rev "R3")
 		(company "Picuino")
 		(comment 1 "License Creative Commons BY-SA 4.0 International")
@@
 	(text "LED LAMP"
 		(exclude_from_sim no)
-		(at 229.362 38.608 0)
+		(at 225.044 38.608 0)
 		(effects
 			(font
@@
 	(text "BATTERY\n(5 AA CELLS)"
 		(exclude_from_sim no)
-		(at 136.652 129.032 0)
+		(at 141.478 127.508 0)
 		(effects
 			(font
@@
 	(text "BOOST CIRCUIT"
 		(exclude_from_sim no)
-		(at 223.012 100.33 0)
+		(at 227.076 100.076 0)
 		(effects
 			(font
@@
 	)
 	(junction
+		(at 209.55 135.89)
+		(diameter 0)
+		(color 0 0 0 0)
+	)
+	(junction
+		(at 199.39 139.7)
+		(diameter 0)
+		(color 0 0 0 0)
+	)
+	(junction
 		(at 246.38 114.3)
 		(diameter 0)
@@
 	(wire
 		(pts
+			(xy 199.39 135.89) (xy 199.39 139.7)
+		)
+		(stroke
+			(width 0)
+			(type default)
+		)
+	)
+	(wire
+		(pts
 			(xy 190.5 114.3) (xy 194.31 114.3)
 		)
@@
 	(wire
 		(pts
-			(xy 233.68 127) (xy 233.68 139.7)
+			(xy 233.68 124.46) (xy 233.68 139.7)
 		)
 		(stroke
@@
 	(wire
 		(pts
+			(xy 209.55 123.19) (xy 209.55 135.89)
+		)
+		(stroke
+			(width 0)
+			(type default)
+		)
+	)
+	(wire
+		(pts
 			(xy 55.88 127) (xy 66.04 127)
 		)
@@
 	(wire
 		(pts
-			(xy 233.68 114.3) (xy 233.68 119.38)
+			(xy 233.68 114.3) (xy 233.68 116.84)
 		)
 		(stroke
@@
 	(wire
 		(pts
-			(xy 194.31 139.7) (xy 215.9 139.7)
+			(xy 199.39 139.7) (xy 215.9 139.7)
+		)
+		(stroke
+			(width 0)
+			(type default)
+		)
+	)
+	(wire
+		(pts
+			(xy 194.31 139.7) (xy 199.39 139.7)
 		)
 		(stroke
@@
 		)
 	)
-	(global_label "+22V"
+	(global_label "LAMP-VCC"
 		(shape input)
 		(at 198.12 50.8 180)
@@
 		)
 		(property "Intersheetrefs" "${INTERSHEET_REFS}"
-			(at 190.709 50.8 0)
+			(at 185.7499 50.8 0)
 			(effects
 				(font
@@
 	(global_label "BOOST_G"
 		(shape input)
-		(at 209.55 135.89 180)
+		(at 209.55 123.19 180)
 		(fields_autoplaced yes)
 		(effects
@@
 		)
 		(property "Intersheetrefs" "${INTERSHEET_REFS}"
-			(at 198.8733 135.89 0)
+			(at 198.8733 123.19 0)
 			(effects
 				(font
@@
 		)
 	)
-	(global_label "+22V"
+	(global_label "LAMP-VCC"
 		(shape input)
 		(at 256.54 114.3 0)
@@
 		)
 		(property "Intersheetrefs" "${INTERSHEET_REFS}"
-			(at 263.951 114.3 0)
+			(at 268.9101 114.3 0)
 			(effects
 				(font
@@
 		(on_board yes)
 		(dnp no)
-		(fields_autoplaced yes)
 		(property "Reference" "L1"
-			(at 204.47 105.41 90)
+			(at 204.216 106.68 90)
 			(effects
 				(font
@@
 			)
 		)
+		(property "Description" "1A"
+			(at 204.47 116.84 90)
+			(effects
+				(font
+					(size 1.905 1.905)
+				)
+			)
+		)
+		(pin ""
+		)
+		(pin ""
+		)
+		(instances
+			(project ""
+				(path "/0802b409-560a-4d90-83f0-c2be7b28d153"
+					(reference "L1")
+					(unit 1)
+				)
+			)
+		)
+	)
+	(symbol
+		(lib_name "resistencia_2")
+		(lib_id "simbolos-electronicos:resistencia")
+		(at 199.39 135.89 90)
+		(unit 1)
+		(exclude_from_sim no)
+		(in_bom yes)
+		(on_board yes)
+		(dnp no)
+		(fields_autoplaced yes)
+		(property "Reference" "R3"
+			(at 204.47 128.1163 90)
+			(effects
+				(font
+					(size 1.905 1.905)
+				)
+			)
+		)
+		(property "Value" "10K"
+			(at 204.47 131.9263 90)
+			(effects
+				(font
+					(size 1.905 1.905)
+				)
+			)
+		)
+		(property "Footprint" ""
+			(at 201.93 133.35 0)
+			(effects
+				(font
+					(size 1.27 1.27)
+				)
+				(hide yes)
+			)
+		)
+		(property "Datasheet" ""
+			(at 201.93 133.35 0)
+			(effects
+				(font
+					(size 1.27 1.27)
+				)
+				(hide yes)
+			)
+		)
 		(property "Description" ""
-			(at 209.55 114.3 0)
+			(at 199.39 135.89 0)
 			(effects
 				(font
@@
 		)
 		(instances
-			(project ""
+			(project "stroboscope"
 				(path "/0802b409-560a-4d90-83f0-c2be7b28d153"
-					(reference "L1")
+					(reference "R3")
 					(unit 1)
 				)
@@
 	(symbol
 		(lib_id "simbolos-electronicos:condensador")
-		(at 233.68 119.38 0)
+		(at 233.68 116.84 0)
 		(unit 1)
 		(exclude_from_sim no)
@@
 		(dnp no)
 		(property "Reference" "C2"
-			(at 229.87 122.2374 0)
+			(at 229.87 119.6974 0)
 			(effects
 				(font
@@
 		)
 		(property "Value" "1000uF"
-			(at 229.87 125.3998 0)
+			(at 229.87 122.8598 0)
 			(effects
 				(font
@@
 		)
 		(property "Footprint" ""
-			(at 234.95 121.92 0)
+			(at 234.95 119.38 0)
 			(effects
 				(font
@@
 		)
 		(property "Datasheet" ""
-			(at 234.95 121.92 0)
+			(at 234.95 119.38 0)
 			(effects
 				(font
@@
 			)
 		)
-		(property "Description" ""
-			(at 233.68 119.38 0)
+		(property "Description" "35V"
+			(at 226.822 125.984 0)
 			(effects
 				(font
-					(size 1.27 1.27)
+					(size 1.905 1.905)
 				)
-				(hide yes)
 			)
 		)
@@
 		(dnp no)
 		(fields_autoplaced yes)
-		(property "Reference" "R4"
+		(property "Reference" "R5"
 			(at 248.92 132.7149 0)
 			(effects
@@
 			(project "stroboscope"
 				(path "/0802b409-560a-4d90-83f0-c2be7b28d153"
-					(reference "R4")
+					(reference "R5")
 					(unit 1)
 				)
@@
 		(dnp no)
 		(fields_autoplaced yes)
-		(property "Reference" "R3"
+		(property "Reference" "R4"
 			(at 248.92 120.0149 0)
 			(effects
@@
 			(project "stroboscope"
 				(path "/0802b409-560a-4d90-83f0-c2be7b28d153"
-					(reference "R3")
+					(reference "R4")
 					(unit 1)
 				)
@@
 			(effects
 				(font
-					(size 1.27 1.27)
+					(size 1.905 1.905)
 				)
 				(justify left)
 			)
 		)
-		(pin "LAMP-GATE" bidirectional
+		(pin "LAMP-ON" bidirectional
 			(at 203.2 58.42 180)
 			(effects
 				(font
-					(size 1.27 1.27)
+					(size 1.905 1.905)
 				)
 				(justify left)
@@
 			(effects
 				(font
-					(size 1.27 1.27)
+					(size 1.905 1.905)
 				)
 				(justify left)
