File: source/electric/electric-simbolos-nombres/electric-nombres.kicad_sch (KiCad schematic)
At the start: 49 parts

Commit message: 17/03/2025 Update
Parts:
- removed CP2: CopyRight, symbol simbolos-electricos:CopyRight
- removed M? (x8): marco_2, symbol electric-symbols-names-rescue:marco_2-simbolos
- removed M? (x39): marco_1, symbol electric-symbols-names-rescue:marco_1-simbolos
- removed M?: marco, symbol electric-symbols-names-rescue:marco_1-simbolos
- added CP1: CopyRight, symbol simbolos-electricos:CopyRight
- added M? (x40): marco_1, symbol electric-simbolos-nombres-rescue:marco_1-simbolos
- added M? (x8): marco_2, symbol electric-simbolos-nombres-rescue:marco_2-simbolos
Other:
- note added: "ALTAVOZ"
- note added: "ALTERNADOR"
- note added: "AMPERÍMETRO"
- note added: "AMPLIFICADOR OPERACIONAL"
- note added: "BOBINA"
- note added: "BOMBILLA"
- note added: "CABLES CON CONEXIÓN"
- note added: "CABLES SIN CONEXIÓN"
- note added: "CONDENSADOR"
- note added: "CONDENSADOR POLARIZADO"
- note added: "CONECTOR"
- note added: "CONEXIÓN A MASA"
- note added: "CONEXIÓN A TIERRA"
- note added: "CONMUTADOR"
- note added: "CONTACTO DE RELÉ"
- note added: "DIODO"
- note added: "DIODO LED"
- note added: "FINAL DE CARRERA"
- note added: "FUSIBLE"
- note added: "INTERRUPTOR"
- note added: "PILA"
- note added: "POTENCIÓMETRO"
- note added: "PUERTA AND"
- note added: "PUERTA NAND"
- note added: "PUERTA NOR"
- note added: "PUERTA NOT"
- note added: "PUERTA OR"
- note added: "PUERTA XOR"
- note added: "PULSADOR NORMALMENTE ABIERTO"
- note added: "PULSADOR NORMALMENTE CERRADO"
- note added: "RELÉ"
- note added: "RESISTENCIA"
- note added: "RESISTENCIA LDR"
- note added: "RESISTENCIA NTC"
- note added: "TRANSFOR- MADOR"
- note added: "TRANSISTOR NPN"
- note added: "TRANSISTOR PNP"
- note added: "VOLTÍMETRO"
- note added: "ZUMBADOR"
- note removed: "A.C. GENERATOR"
- note removed: "AMMETER"
- note removed: "AND GATE"
- note removed: "BATTERY"
- note removed: "BULB LAMP"
- note removed: "BUZZER"
- note removed: "CAPACITOR"
- note removed: "CHASSIS GROUND CONNECTOR"
- note removed: "CONNECTOR"
- note removed: "DIODE"
- note removed: "DOUBLE THROW SWITCH"
- note removed: "EARTH GROUND CONNECTOR"
- note removed: "FUSE"
- note removed: "INDUCTOR/COIL"
- note removed: "LDR RESISTOR"
- note removed: "LIGHT EMITTING DIODE (LED)"
- note removed: "LIMIT SWITCH"
- note removed: "LOUDSPEAKER"
- note removed: "NAND GATE"
- note removed: "NOR GATE"
- note removed: "NORMALLY CLOSED PUSH BUTTON"
- note removed: "NORMALLY OPEN PUSH BUTTON"
- note removed: "NOT GATE"
- note removed: "NPN TRANSISTOR"
- note removed: "NTC RESISTOR"
- note removed: "OPERATIONAL AMPLIFIER"
- note removed: "OR GATE"
- note removed: "PNP TRANSISTOR"
- note removed: "POLARIZED CAPACITOR"
- note removed: "POTENTIOMETER"
- note removed: "RELAY"
- note removed: "RELAY CONTACT"
- note removed: "RESISTOR"
- note removed: "SWITCH"
- note removed: "TRANSFORMER"
- note removed: "VOLTMETER"
- note removed: "WIRES WITH CONNECTION"
- note removed: "WIRES WITHOUT CONNECTION"
- note removed: "XOR GATE"

Commit message: 20/04/2026 Update
Parts:
- added M3: marco_1, symbol electric-simbolos-nombres-rescue:marco_1-simbolos
- CP1: License CC BY-SA 4.0 -> Licencia CC BY-SA 4.0
Other:
- note added: "BORNA DE CONEXIÓN"
