File: source/electric/electric-simbolos-nombres/electric-simbolos-nombres.kicad_sch (KiCad schematic)
At the start: 88 parts, among them J1 conector, K1 CONTACTO, K1 RELE, M1 MOTOR, Q1 TRANSISTOR, Q2 TRANSISTOR, U1 OA, U1 logic_and, U2 logic_and, U3 logic_and, U4 logic_and, U5 logic_and, U6 logic_and

Commit message: 17/03/2025 Update
Parts:
- removed CP1: CopyRight, symbol simbolos-electricos:CopyRight
- removed R1: RESISTENCIA, symbol electric-symbols-names-rescue:resistencia-simbolos
- removed R5: resistencia, symbol simbolos-electricos:resistencia_2
- removed U1: OA, symbol simbolos-electricos:OA
- added CP2: CopyRight, symbol simbolos-electricos:CopyRight
- added R1: RESISTENCIA, symbol electric-simbolos-nombres-rescue:resistencia-simbolos
- added R5: resistencia, symbol simbolos-electricos:resistencia
- added U1: AO, symbol simbolos-electricos:AO
- A: symbol electric-symbols-names-rescue:amperimetro-simbolos -> electric-simbolos-nombres-rescue:amperimetro-simbolos
- B1: symbol electric-symbols-names-rescue:lampara-simbolos -> electric-simbolos-nombres-rescue:lampara-simbolos
- C1: renamed from C2; symbol electric-symbols-names-rescue:condensador-simbolos -> electric-simbolos-nombres-rescue:condensador-simbolos
- C2: renamed from C1; symbol electric-symbols-names-rescue:condensador_pol-simbolos -> electric-simbolos-nombres-rescue:condensador_pol-simbolos
- D1: symbol electric-symbols-names-rescue:diodo-simbolos -> electric-simbolos-nombres-rescue:diodo-simbolos
- D2: symbol electric-symbols-names-rescue:diodo_led-simbolos -> electric-simbolos-nombres-rescue:diodo_led-simbolos
- F1: symbol electric-symbols-names-rescue:fusible-simbolos -> electric-simbolos-nombres-rescue:fusible-simbolos
- J1: symbol electric-symbols-names-rescue:conector-simbolos -> electric-simbolos-nombres-rescue:conector-simbolos
- K1: symbol electric-symbols-names-rescue:rele_contacto-simbolos -> electric-simbolos-nombres-rescue:rele_contacto-simbolos
- K1: symbol electric-symbols-names-rescue:rele-simbolos -> electric-simbolos-nombres-rescue:rele-simbolos
- L1: symbol electric-symbols-names-rescue:inductancia-simbolos -> electric-simbolos-nombres-rescue:inductancia-simbolos
- M1: symbol electric-symbols-names-rescue:motor-simbolos -> electric-simbolos-nombres-rescue:motor-simbolos
- M?: symbol electric-symbols-names-rescue:marco_2-simbolos -> electric-simbolos-nombres-rescue:marco_2-simbolos; Campo4 LOGIC GATES -> PUERTAS LÓGICAS; Campo5 SYMBOL -> SÍMBOLO; Campo6 LETTER -> LETRA; Campo7 NAME -> NOMBRE
- M? (x40): symbol electric-symbols-names-rescue:marco_1-simbolos -> electric-simbolos-nombres-rescue:marco_1-simbolos
- M?: symbol electric-symbols-names-rescue:marco_2-simbolos -> electric-simbolos-nombres-rescue:marco_2-simbolos; Campo4 GENERATORS -> GENERADORES; Campo5 SYMBOL -> SÍMBOLO; Campo6 LETTER -> LETRA; Campo7 NAME -> NOMBRE
- M?: symbol electric-symbols-names-rescue:marco_2-simbolos -> electric-simbolos-nombres-rescue:marco_2-simbolos; Campo4 CONTROL COMPONENTS -> ELEMENTOS DE CONTROL; Campo5 SYMBOL -> SÍMBOLO; Campo6 LETTER -> LETRA; Campo7 NAME -> NOMBRE
- M?: symbol electric-symbols-names-rescue:marco_2-simbolos -> electric-simbolos-nombres-rescue:marco_2-simbolos; Campo4 ELECTRICAL LOADS -> RECEPTORES; Campo5 SYMBOL -> SÍMBOLO; Campo6 LETTER -> LETRA; Campo7 NAME -> NOMBRE
- M?: symbol electric-symbols-names-rescue:marco_2-simbolos -> electric-simbolos-nombres-rescue:marco_2-simbolos; Campo4 SENSORS -> SENSORES; Campo5 SYMBOL -> SÍMBOLO; Campo6 LETTER -> LETRA; Campo7 NAME -> NOMBRE
- M?: symbol electric-symbols-names-rescue:marco_2-simbolos -> electric-simbolos-nombres-rescue:marco_2-simbolos; Campo4 CONDUCTORS -> CONDUCTORES; Campo5 SYMBOL -> SÍMBOLO; Campo6 LETTER -> LETRA; Campo7 NAME -> NOMBRE
- M?: symbol electric-symbols-names-rescue:marco_2-simbolos -> electric-simbolos-nombres-rescue:marco_2-simbolos; Campo4 MEASURING INSTRUMENTS -> APARATOS DE MEDIDA; Campo5 SYMBOL -> SÍMBOLO; Campo6 LETTER -> LETRA; Campo7 NAME -> NOMBRE
- M?: symbol electric-symbols-names-rescue:marco_2-simbolos -> electric-simbolos-nombres-rescue:marco_2-simbolos; Campo4 ELECTRONIC COMPONENTS -> COMPONENTES ELECTRÓNICOS; Campo5 SYMBOL -> SÍMBOLO; Campo6 LETTER -> LETRA; Campo7 NAME -> NOMBRE
- S1: symbol electric-symbols-names-rescue:switch-simbolos -> electric-simbolos-nombres-rescue:switch-simbolos
- S2: symbol electric-symbols-names-rescue:selector-simbolos -> electric-simbolos-nombres-rescue:selector-simbolos
- S3: symbol electric-symbols-names-rescue:pulsador_na-simbolos -> electric-simbolos-nombres-rescue:pulsador_na-simbolos
- S4: symbol electric-symbols-names-rescue:pulsador_nc-simbolos -> electric-simbolos-nombres-rescue:pulsador_nc-simbolos
- S5: symbol electric-symbols-names-rescue:final_carrera-simbolos -> electric-simbolos-nombres-rescue:final_carrera-simbolos
- U1: symbol electric-symbols-names-rescue:logic_and-simbolos -> electric-simbolos-nombres-rescue:logic_and-simbolos
- U2: symbol electric-symbols-names-rescue:logic_or-simbolos -> electric-simbolos-nombres-rescue:logic_or-simbolos
- U3: symbol electric-symbols-names-rescue:logic_not-simbolos -> electric-simbolos-nombres-rescue:logic_not-simbolos
- U4: symbol electric-symbols-names-rescue:logic_nand-simbolos -> electric-simbolos-nombres-rescue:logic_nand-simbolos
- U5: symbol electric-symbols-names-rescue:logic_nor-simbolos -> electric-simbolos-nombres-rescue:logic_nor-simbolos
- U6: symbol electric-symbols-names-rescue:logic_xor-simbolos -> electric-simbolos-nombres-rescue:logic_xor-simbolos
- V2: symbol electric-symbols-names-rescue:generador-simbolos -> electric-simbolos-nombres-rescue:generador-simbolos
- V?: value CONNECTION -> CONEXIÓN; symbol electric-symbols-names-rescue:masa-simbolos -> electric-simbolos-nombres-rescue:masa-simbolos
- V?: value CONNECTION -> CONEXIÓN
Other:
- sheet Component Symbols renamed Simbolos de componentes
- sheet Component names renamed Nombres de componentes
- sheet Nombres de componentes: file electric-names.kicad_sch -> electric-nombres.kicad_sch
- sheet Simbolos de componentes: file electric-symbols.kicad_sch -> electric-simbolos.kicad_sch
- note added: "ALTAVOZ"
- note added: "ALTERNADOR"
- note added: "AMPERÍMETRO"
- note added: "AMPLIFICADOR OPERACIONAL"
- note added: "BOBINA"
- note added: "BOMBILLA"
- note added: "CABLES CON CONEXIÓN"
- note added: "CABLES SIN CONEXIÓN"
- note added: "CONDENSADOR"
- note added: "CONDENSADOR POLARIZADO"
- note added: "CONECTOR"
- note added: "CONEXIÓN A MASA"
- note added: "CONEXIÓN A TIERRA"
- note added: "CONMUTADOR"
- note added: "CONTACTO DE RELÉ"
- note added: "DIODO"
- note added: "DIODO LED"
- note added: "FINAL DE CARRERA"
- note added: "FUSIBLE"
- note added: "INTERRUPTOR"
- note added: "PILA"
- note added: "POTENCIÓMETRO"
- note added: "PUERTA AND"
- note added: "PUERTA NAND"
- note added: "PUERTA NOR"
- note added: "PUERTA NOT"
- note added: "PUERTA OR"
- note added: "PUERTA XOR"
- note added: "PULSADOR NORMALMENTE ABIERTO"
- note added: "PULSADOR NORMALMENTE CERRADO"
- note added: "RELÉ"
- note added: "RESISTENCIA"
- note added: "RESISTENCIA LDR"
- note added: "RESISTENCIA NTC"
- note added: "TRANSFOR- MADOR"
- note added: "TRANSISTOR NPN"
- note added: "TRANSISTOR PNP"
- note added: "VOLTÍMETRO"
- note added: "ZUMBADOR"
- note removed: "A.C. GENERATOR"
- note removed: "AMMETER"
- note removed: "AND GATE"
- note removed: "BATTERY"
- note removed: "BUZZER"
- note removed: "CAPACITOR"
- note removed: "CHASSIS GROUND CONNECTOR"
- note removed: "CONNECTOR"
- note removed: "DIODE"
- note removed: "DOUBLE THROW SWITCH"
- note removed: "EARTH GROUND CONNECTOR"
- note removed: "FUSE"
- note removed: "INCANDESCENT LAMP"
- note removed: "INDUCTOR"
- note removed: "LDR RESISTOR"
- note removed: "LIGHT EMITTING DIODE (LED)"
- note removed: "LIMIT SWITCH"
- note removed: "LOUDSPEAKER"
- note removed: "NAND GATE"
- note removed: "NOR GATE"
- note removed: "NORMALLY CLOSED PUSHBUTTON"
- note removed: "NORMALLY OPEN PUSHBUTTON"
- note removed: "NOT GATE"
- note removed: "NPN TRANSISTOR"
- note removed: "NTC RESISTOR"
- note removed: "OPERATIONAL AMPLIFIER"
- note removed: "OR GATE"
- note removed: "PNP TRANSISTOR"
- note removed: "POLARIZED CAPACITOR"
- note removed: "POTENTIOMETER"
- note removed: "RELAY"
- note removed: "RELAY CONTACT"
- note removed: "RESISTOR"
- note removed: "SWITCH"
- note removed: "TRANSFORMER"
- note removed: "VOLTMETER"
- note removed: "WIRES WITH CONNECTION"
- note removed: "WIRES WITHOUT CONNECTION"
- note removed: "XOR GATE"

Commit message: 18/03/2025 Update
Parts:
- removed R1: RESISTENCIA, symbol electric-simbolos-nombres-rescue:resistencia-simbolos
- added R1: resistencia, symbol simbolos-electricos:resistencia_2
- renumbered R5 to R1
Changed lines of the file:
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@@
 		(on_board yes)
 		(dnp no)
-		(fields_autoplaced yes)
-		(property "Reference" "R5"
-			(at 16.51 125.095 90)
+		(property "Reference" "R1"
+			(at 32.766 133.35 90)
 			(effects
 				(font
 					(size 2.54 2.54)
 				)
-				(hide yes)
 			)
 		)
@@
 			(project ""
 				(path "/275d908d-d95f-4e76-9103-a82879596f4e"
-					(reference "R5")
+					(reference "R1")
 					(unit 1)
 				)
@@
 	)
 	(symbol
-		(lib_id "electric-simbolos-nombres-rescue:resistencia-simbolos")
+		(lib_id "simbolos-electricos:resistencia_2")
 		(at 11.43 137.16 90)
 		(unit 1)
@@
 		(on_board yes)
 		(dnp no)
+		(fields_autoplaced yes)
 		(property "Reference" "R1"
-			(at 32.766 133.35 90)
+			(at 16.51 132.08 90)
 			(effects
 				(font
 					(size 2.54 2.54)
 				)
+				(hide yes)
 			)
 		)
-		(property "Value" "RESISTENCIA"
-			(at -6.985 137.16 90)
+		(property "Value" "resistencia"
+			(at 17.145 139.7 90)
 			(effects
 				(font
-					(size 2.54 2.54)
+					(size 1.27 1.27)
 				)
-				(justify left)
 				(hide yes)
 			)

Commit message: 28/07/2025 Update
Parts:
- renumbered U1 to U2, U2 to U3, U3 to U4, U4 to U5, U5 to U6, U6 to U7
Changed lines of the file:
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@@
 		(on_board yes)
 		(dnp no)
-		(property "Reference" "U1"
+		(property "Reference" "U2"
 			(at 167.64 194.31 0)
 			(effects
@@
 			(project "electric-simbolos-nombres"
 				(path "/275d908d-d95f-4e76-9103-a82879596f4e"
-					(reference "U1")
+					(reference "U2")
 					(unit 1)
 				)
@@
 		(on_board yes)
 		(dnp no)
-		(property "Reference" "U2"
+		(property "Reference" "U3"
 			(at 167.64 209.55 0)
 			(effects
@@
 			(project "electric-simbolos-nombres"
 				(path "/275d908d-d95f-4e76-9103-a82879596f4e"
-					(reference "U2")
+					(reference "U3")
 					(unit 1)
 				)
@@
 		(on_board yes)
 		(dnp no)
-		(property "Reference" "U3"
+		(property "Reference" "U4"
 			(at 167.64 224.79 0)
 			(effects
@@
 			(project "electric-simbolos-nombres"
 				(path "/275d908d-d95f-4e76-9103-a82879596f4e"
-					(reference "U3")
+					(reference "U4")
 					(unit 1)
 				)
@@
 		(on_board yes)
 		(dnp no)
-		(property "Reference" "U4"
+		(property "Reference" "U5"
 			(at 167.64 240.03 0)
 			(effects
@@
 			(project "electric-simbolos-nombres"
 				(path "/275d908d-d95f-4e76-9103-a82879596f4e"
-					(reference "U4")
+					(reference "U5")
 					(unit 1)
 				)
@@
 		(on_board yes)
 		(dnp no)
-		(property "Reference" "U5"
+		(property "Reference" "U6"
 			(at 167.64 255.27 0)
 			(effects
@@
 			(project "electric-simbolos-nombres"
 				(path "/275d908d-d95f-4e76-9103-a82879596f4e"
-					(reference "U5")
+					(reference "U6")
 					(unit 1)
 				)
@@
 		(on_board yes)
 		(dnp no)
-		(property "Reference" "U6"
+		(property "Reference" "U7"
 			(at 167.64 270.51 0)
 			(effects
@@
 			(project "electric-simbolos-nombres"
 				(path "/275d908d-d95f-4e76-9103-a82879596f4e"
-					(reference "U6")
+					(reference "U7")
 					(unit 1)
 				)

Commit message: 20/04/2026 Update
Parts:
- added M2: marco_1, symbol electric-simbolos-nombres-rescue:marco_1-simbolos
- added X1: ~, symbol simbolos-electricos:Borna
- CP2: License CC BY-SA 4.0 -> Licencia CC BY-SA 4.0
- renumbered C2 to C1, C1 to C2
Other:
- note added: "BORNA DE CONEXIÓN"
