File: source/electric/electric-simbolos-nombres/electric-simbolos.kicad_sch (KiCad schematic)
At the start: 88 parts, among them J1 conector, K1 CONTACTO, K1 RELE, M1 MOTOR, Q1 TRANSISTOR, Q2 TRANSISTOR, U1 OA, U1 logic_and, U2 logic_and, U3 logic_and, U4 logic_and, U5 logic_and, U6 logic_and

Commit message: 17/03/2025 Update
Parts:
- removed A: amperimetro, symbol electric-symbols-names-rescue:amperimetro-simbolos
- removed B1: LÁMPARA, symbol electric-symbols-names-rescue:lampara-simbolos
- removed C1: CONDENSADOR, symbol electric-symbols-names-rescue:condensador_pol-simbolos
- removed C2: CONDENSADOR, symbol electric-symbols-names-rescue:condensador-simbolos
- removed CP1: CopyRight, symbol simbolos-electricos:CopyRight
- removed D1: DIODO, symbol electric-symbols-names-rescue:diodo-simbolos
- removed D2: DIODO LED, symbol electric-symbols-names-rescue:diodo_led-simbolos
- removed F1: FUSIBLE, symbol electric-symbols-names-rescue:fusible-simbolos
- removed J1: conector, symbol electric-symbols-names-rescue:conector-simbolos
- removed K1: CONTACTO, symbol electric-symbols-names-rescue:rele_contacto-simbolos
- removed K1: RELE, symbol electric-symbols-names-rescue:rele-simbolos
- removed L1: INDUCTANCIA, symbol electric-symbols-names-rescue:inductancia-simbolos
- removed M1: MOTOR, symbol electric-symbols-names-rescue:motor-simbolos
- removed M? (x8): marco_2, symbol electric-symbols-names-rescue:marco_2-simbolos
- removed M? (x39): marco_1, symbol electric-symbols-names-rescue:marco_1-simbolos
- removed M?: marco, symbol electric-symbols-names-rescue:marco_1-simbolos
- removed R1: RESISTENCIA, symbol electric-symbols-names-rescue:resistencia-simbolos
- removed R5: resistencia, symbol simbolos-electricos:resistencia_2
- removed S1: INTERRUPTOR, symbol electric-symbols-names-rescue:switch-simbolos
- removed S2: CONMUTADOR, symbol electric-symbols-names-rescue:selector-simbolos
- removed S3: PULSADOR, symbol electric-symbols-names-rescue:pulsador_na-simbolos
- removed S4: PULSADOR, symbol electric-symbols-names-rescue:pulsador_nc-simbolos
- removed S5: FINAL DE, symbol electric-symbols-names-rescue:final_carrera-simbolos
- removed U1: logic_and, symbol electric-symbols-names-rescue:logic_and-simbolos
- removed U1: OA, symbol simbolos-electricos:OA
- removed U2: logic_and, symbol electric-symbols-names-rescue:logic_or-simbolos
- removed U3: logic_and, symbol electric-symbols-names-rescue:logic_not-simbolos
- removed U4: logic_and, symbol electric-symbols-names-rescue:logic_nand-simbolos
- removed U5: logic_and, symbol electric-symbols-names-rescue:logic_nor-simbolos
- removed U6: logic_and, symbol electric-symbols-names-rescue:logic_xor-simbolos
- removed V2: GENERADOR, symbol electric-symbols-names-rescue:generador-simbolos
- removed V?: CONNECTION, symbol electric-symbols-names-rescue:masa-simbolos
- removed V?: CONNECTION, symbol simbolos-electricos:tierra
- added A: amperimetro, symbol electric-simbolos-nombres-rescue:amperimetro-simbolos
- added B1: LÁMPARA, symbol electric-simbolos-nombres-rescue:lampara-simbolos
- added C1: CONDENSADOR, symbol electric-simbolos-nombres-rescue:condensador-simbolos
- added C2: CONDENSADOR, symbol electric-simbolos-nombres-rescue:condensador_pol-simbolos
- added CP3: CopyRight, symbol simbolos-electricos:CopyRight
- added D1: DIODO, symbol electric-simbolos-nombres-rescue:diodo-simbolos
- added D2: DIODO LED, symbol electric-simbolos-nombres-rescue:diodo_led-simbolos
- added F1: FUSIBLE, symbol electric-simbolos-nombres-rescue:fusible-simbolos
- added J1: conector, symbol electric-simbolos-nombres-rescue:conector-simbolos
- added K1: RELE, symbol electric-simbolos-nombres-rescue:rele-simbolos
- added K1: CONTACTO, symbol electric-simbolos-nombres-rescue:rele_contacto-simbolos
- added L1: INDUCTANCIA, symbol electric-simbolos-nombres-rescue:inductancia-simbolos
- added M1: MOTOR, symbol electric-simbolos-nombres-rescue:motor-simbolos
- added M? (x39): marco_1, symbol electric-simbolos-nombres-rescue:marco_1-simbolos
- added M? (x8): marco_2, symbol electric-simbolos-nombres-rescue:marco_2-simbolos
- added M?: marco, symbol electric-simbolos-nombres-rescue:marco_1-simbolos
- added R1: RESISTENCIA, symbol electric-simbolos-nombres-rescue:resistencia-simbolos
- added R6: resistencia, symbol simbolos-electricos:resistencia
- added S1: INTERRUPTOR, symbol electric-simbolos-nombres-rescue:switch-simbolos
- added S2: CONMUTADOR, symbol electric-simbolos-nombres-rescue:selector-simbolos
- added S3: PULSADOR, symbol electric-simbolos-nombres-rescue:pulsador_na-simbolos
- added S4: PULSADOR, symbol electric-simbolos-nombres-rescue:pulsador_nc-simbolos
- added S5: FINAL DE, symbol electric-simbolos-nombres-rescue:final_carrera-simbolos
- added U1: AO, symbol simbolos-electricos:AO
- added U1: logic_and, symbol simbolos-electricos:logic_and
- added U2: logic_or, symbol simbolos-electricos:logic_or
- added U3: logic_not, symbol simbolos-electricos:logic_not
- added U4: logic_nand, symbol simbolos-electricos:logic_nand
- added U5: logic_nor, symbol simbolos-electricos:logic_nor
- added U6: logic_xor, symbol simbolos-electricos:logic_xor
- added V2: GENERADOR, symbol electric-simbolos-nombres-rescue:generador-simbolos
- added V?: CONEXIÓN, symbol simbolos-electricos:tierra
- added V?: CONEXIÓN, symbol electric-simbolos-nombres-rescue:masa-simbolos
Other:
- removed sheet Component Symbols
- removed sheet Component names
- note removed: "A.C. GENERATOR"
- note removed: "AMMETER"
- note removed: "AND GATE"
- note removed: "BATTERY"
- note removed: "BUZZER"
- note removed: "CAPACITOR"
- note removed: "CHASSIS GROUND CONNECTOR"
- note removed: "CONNECTOR"
- note removed: "DIODE"
- note removed: "DOUBLE THROW SWITCH"
- note removed: "EARTH GROUND CONNECTOR"
- note removed: "FUSE"
- note removed: "INCANDESCENT LAMP"
- note removed: "INDUCTOR"
- note removed: "LDR RESISTOR"
- note removed: "LIGHT EMITTING DIODE (LED)"
- note removed: "LIMIT SWITCH"
- note removed: "LOUDSPEAKER"
- note removed: "MOTOR"
- note removed: "NAND GATE"
- note removed: "NOR GATE"
- note removed: "NORMALLY CLOSED PUSHBUTTON"
- note removed: "NORMALLY OPEN PUSHBUTTON"
- note removed: "NOT GATE"
- note removed: "NPN TRANSISTOR"
- note removed: "NTC RESISTOR"
- note removed: "OPERATIONAL AMPLIFIER"
- note removed: "OR GATE"
- note removed: "PNP TRANSISTOR"
- note removed: "POLARIZED CAPACITOR"
- note removed: "POTENTIOMETER"
- note removed: "RELAY"
- note removed: "RELAY CONTACT"
- note removed: "RESISTOR"
- note removed: "SWITCH"
- note removed: "TRANSFORMER"
- note removed: "VOLTMETER"
- note removed: "WIRES WITH CONNECTION"
- note removed: "WIRES WITHOUT CONNECTION"
- note removed: "XOR GATE"

Commit message: 18/03/2025 Update
Parts:
- removed R1: RESISTENCIA, symbol electric-simbolos-nombres-rescue:resistencia-simbolos
- added R1: resistencia, symbol simbolos-electricos:resistencia_2
- renumbered R6 to R1
Changed lines of the file:
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@@
 		(on_board yes)
 		(dnp no)
-		(fields_autoplaced yes)
-		(property "Reference" "R6"
-			(at 16.51 124.46 90)
+		(property "Reference" "R1"
+			(at 33.02 133.604 90)
 			(effects
 				(font
 					(size 2.54 2.54)
 				)
-				(hide yes)
 			)
 		)
@@
 			(project ""
 				(path "/275d908d-d95f-4e76-9103-a82879596f4e/00000000-0000-0000-0000-00005bc9ce01"
-					(reference "R6")
+					(reference "R1")
 					(unit 1)
 				)
@@
 	)
 	(symbol
-		(lib_id "electric-simbolos-nombres-rescue:resistencia-simbolos")
-		(at 21.59 137.16 270)
-		(unit 1)
-		(exclude_from_sim no)
-		(in_bom yes)
-		(on_board yes)
-		(dnp no)
-		(property "Reference" "R1"
-			(at 32.766 133.604 90)
-			(effects
-				(font
-					(size 2.54 2.54)
-				)
-			)
-		)
-		(property "Value" "RESISTENCIA"
-			(at 40.005 137.16 90)
-			(effects
-				(font
-					(size 2.54 2.54)
-				)
-				(justify left)
-				(hide yes)
-			)
-		)
-		(property "Footprint" ""
-			(at 19.05 139.7 0)
-			(effects
-				(font
-					(size 1.27 1.27)
-				)
-				(hide yes)
-			)
-		)
-		(property "Datasheet" ""
-			(at 19.05 139.7 0)
-			(effects
-				(font
-					(size 1.27 1.27)
-				)
-				(hide yes)
-			)
-		)
-		(property "Description" ""
-			(at 21.59 137.16 0)
-			(effects
-				(font
-					(size 1.27 1.27)
-				)
-				(hide yes)
-			)
-		)
-		(pin ""
-		)
-		(pin ""
-		)
-		(instances
-			(project ""
-				(path "/275d908d-d95f-4e76-9103-a82879596f4e"
-					(reference "R1")
-					(unit 1)
-				)
-				(path "/275d908d-d95f-4e76-9103-a82879596f4e/00000000-0000-0000-0000-00005bc9ce01"
-					(reference "R1")
-					(unit 1)
-				)
-			)
-		)
-	)
-	(symbol
 		(lib_id "electric-simbolos-nombres-rescue:marco_1-simbolos")
 		(at 72.39 201.93 0)
@@
 					(unit 1)
 				)
+			)
+		)
+	)
+	(symbol
+		(lib_id "simbolos-electricos:resistencia_2")
+		(at 11.43 137.16 90)
+		(unit 1)
+		(exclude_from_sim no)
+		(in_bom yes)
+		(on_board yes)
+		(dnp no)
+		(fields_autoplaced yes)
+		(property "Reference" "R1"
+			(at 16.51 132.08 90)
+			(effects
+				(font
+					(size 2.54 2.54)
+				)
+				(hide yes)
+			)
+		)
+		(property "Value" "resistencia"
+			(at 17.145 139.7 90)
+			(effects
+				(font
+					(size 1.27 1.27)
+				)
+				(hide yes)
+			)
+		)
+		(property "Footprint" ""
+			(at 13.97 134.62 0)
+			(effects
+				(font
+					(size 1.27 1.27)
+				)
+				(hide yes)
+			)
+		)
+		(property "Datasheet" ""
+			(at 13.97 134.62 0)
+			(effects
+				(font
+					(size 1.27 1.27)
+				)
+				(hide yes)
+			)
+		)
+		(property "Description" ""
+			(at 11.43 137.16 0)
+			(effects
+				(font
+					(size 1.27 1.27)
+				)
+				(hide yes)
+			)
+		)
+		(pin ""
+		)
+		(pin ""
+		)
+		(instances
+			(project ""
+				(path "/275d908d-d95f-4e76-9103-a82879596f4e/00000000-0000-0000-0000-00005bc9ce01"
+					(reference "R1")
+					(unit 1)
+				)

Commit message: 28/07/2025 Update
Parts:
- removed U1: AO, symbol simbolos-electricos:AO
- added U1: AO, symbol simbolos-electricos:OA
- U3: renamed from U2; value logic_or -> logic_and; Campo4 (none) -> PUERTA OR
- U4: renamed from U3; value logic_not -> logic_and; Campo4 (none) -> PUERTA NOT
- U5: renamed from U4; value logic_nand -> logic_and; Campo4 (none) -> PUERTA NAND
- U6: renamed from U5; value logic_nor -> logic_and; Campo4 (none) -> PUERTA NOR
- U7: renamed from U6; value logic_xor -> logic_and; Campo4 (none) -> PUERTA XOR
- renumbered U1 to U2
Changed lines of the file:
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@@
 	)
 	(symbol
-		(lib_id "simbolos-electricos:AO")
-		(at 146.685 87.63 0)
-		(unit 1)
-		(exclude_from_sim no)
-		(in_bom yes)
-		(on_board yes)
-		(dnp no)
-		(property "Reference" "U1"
-			(at 167.64 87.63 0)
-			(effects
-				(font
-					(size 2.54 2.54)
-				)
-			)
-		)
-		(property "Value" "AO"
-			(at 151.13 87.63 0)
-			(effects
-				(font
-					(size 1.27 1.27)
-				)
-			)
-		)
-		(property "Footprint" ""
-			(at 146.685 87.63 0)
-			(effects
-				(font
-					(size 1.27 1.27)
-				)
-				(hide yes)
-			)
-		)
-		(property "Datasheet" ""
-			(at 146.685 87.63 0)
-			(effects
-				(font
-					(size 1.27 1.27)
-				)
-				(hide yes)
-			)
-		)
-		(property "Description" ""
-			(at 146.685 87.63 0)
-			(effects
-				(font
-					(size 1.27 1.27)
-				)
-				(hide yes)
-			)
-		)
-		(pin ""
-		)
-		(pin ""
-		)
-		(pin ""
-		)
-		(instances
-			(project "electric-simbolos-nombres"
-				(path "/275d908d-d95f-4e76-9103-a82879596f4e/00000000-0000-0000-0000-00005bc9ce01"
-					(reference "U1")
-					(unit 1)
-				)
-			)
-		)
-	)
-	(symbol
 		(lib_id "electric-simbolos-nombres-rescue:amperimetro-simbolos")
 		(at 16.51 265.43 0)
@@
 		(on_board yes)
 		(dnp no)
-		(property "Reference" "U5"
+		(property "Reference" "U6"
 			(at 167.64 255.27 0)
 			(effects
@@
 			)
 		)
-		(property "Value" "logic_nor"
+		(property "Value" "logic_and"
 			(at 151.13 250.19 0)
 			(effects
@@
 			)
 		)
+		(property "Campo4" "PUERTA NOR"
+			(at 174.625 255.27 0)
+			(effects
+				(font
+					(size 2.54 2.54)
+				)
+				(justify left)
+				(hide yes)
+			)
+		)
 		(pin ""
 		)
@@
 		)
 		(instances
-			(project "electric-simbolos-nombres"
+			(project ""
+				(path "/275d908d-d95f-4e76-9103-a82879596f4e"
+					(reference "U6")
+					(unit 1)
+				)
 				(path "/275d908d-d95f-4e76-9103-a82879596f4e/00000000-0000-0000-0000-00005bc9ce01"
-					(reference "U5")
+					(reference "U6")
 					(unit 1)
 				)
@@
 	)
 	(symbol
+		(lib_id "simbolos-electricos:OA")
+		(at 146.05 87.63 0)
+		(unit 1)
+		(exclude_from_sim no)
+		(in_bom yes)
+		(on_board yes)
+		(dnp no)
+		(property "Reference" "U1"
+			(at 167.64 87.63 0)
+			(effects
+				(font
+					(size 2.54 2.54)
+				)
+			)
+		)
+		(property "Value" "AO"
+			(at 150.495 87.63 0)
+			(effects
+				(font
+					(size 1.27 1.27)
+				)
+				(hide yes)
+			)
+		)
+		(property "Footprint" ""
+			(at 146.05 87.63 0)
+			(effects
+				(font
+					(size 1.27 1.27)
+				)
+				(hide yes)
+			)
+		)
+		(property "Datasheet" ""
+			(at 146.05 87.63 0)
+			(effects
+				(font
+					(size 1.27 1.27)
+				)
+				(hide yes)
+			)
+		)
+		(property "Description" ""
+			(at 146.05 87.63 0)
+			(effects
+				(font
+					(size 1.27 1.27)
+				)
+				(hide yes)
+			)
+		)
+		(pin ""
+		)
+		(pin ""
+		)
+		(pin ""
+		)
+		(instances
+			(project ""
+				(path "/275d908d-d95f-4e76-9103-a82879596f4e"
+					(reference "U1")
+					(unit 1)
+				)
+				(path "/275d908d-d95f-4e76-9103-a82879596f4e/00000000-0000-0000-0000-00005bc9ce01"
+					(reference "U1")
+					(unit 1)
+				)
+			)
+		)
+	)
+	(symbol
 		(lib_id "simbolos-electricos:resistencia")
 		(at 11.43 129.54 90)
@@
 		(on_board yes)
 		(dnp no)
-		(property "Reference" "U6"
+		(property "Reference" "U7"
 			(at 167.64 270.51 0)
 			(effects
@@
 			)
 		)
-		(property "Value" "logic_xor"
+		(property "Value" "logic_and"
 			(at 151.13 265.43 0)
 			(effects
@@
 			)
 		)
+		(property "Campo4" "PUERTA XOR"
+			(at 174.625 270.51 0)
+			(effects
+				(font
+					(size 2.54 2.54)
+				)
+				(justify left)
+				(hide yes)
+			)
+		)
 		(pin ""
 		)
@@
 		)
 		(instances
-			(project "electric-simbolos-nombres"
+			(project ""
+				(path "/275d908d-d95f-4e76-9103-a82879596f4e"
+					(reference "U7")
+					(unit 1)
+				)
 				(path "/275d908d-d95f-4e76-9103-a82879596f4e/00000000-0000-0000-0000-00005bc9ce01"
-					(reference "U6")
+					(reference "U7")
 					(unit 1)
 				)
@@
 		(on_board yes)
 		(dnp no)
-		(property "Reference" "U1"
+		(property "Reference" "U2"
 			(at 167.64 194.31 0)
 			(effects
@@
 			)
 		)
+		(property "Campo4" ""
+			(at 174.625 194.31 0)
+			(effects
+				(font
+					(size 2.54 2.54)
+				)
+				(justify left)
+			)
+		)
 		(pin ""
 		)
@@
 		)
 		(instances
-			(project "electric-simbolos-nombres"
+			(project ""
+				(path "/275d908d-d95f-4e76-9103-a82879596f4e"
+					(reference "U2")
+					(unit 1)
+				)
 				(path "/275d908d-d95f-4e76-9103-a82879596f4e/00000000-0000-0000-0000-00005bc9ce01"
-					(reference "U1")
+					(reference "U2")
 					(unit 1)
 				)
@@
 		(on_board yes)
 		(dnp no)
-		(property "Reference" "U3"
+		(property "Reference" "U4"
 			(at 167.64 224.79 0)
 			(effects
@@
 			)
 		)
-		(property "Value" "logic_not"
-			(at 152.4 219.71 0)
+		(property "Value" "logic_and"
+			(at 151.13 219.71 0)
 			(effects
 				(font
@@
 			)
 		)
+		(property "Campo4" "PUERTA NOT"
+			(at 174.625 224.79 0)
+			(effects
+				(font
+					(size 2.54 2.54)
+				)
+				(justify left)
+				(hide yes)
+			)
+		)
 		(pin ""
 		)
@@
 		)
 		(instances
-			(project "electric-simbolos-nombres"
+			(project ""
+				(path "/275d908d-d95f-4e76-9103-a82879596f4e"
+					(reference "U4")
+					(unit 1)
+				)
 				(path "/275d908d-d95f-4e76-9103-a82879596f4e/00000000-0000-0000-0000-00005bc9ce01"
-					(reference "U3")
+					(reference "U4")
 					(unit 1)
 				)
@@
 		(on_board yes)
 		(dnp no)
-		(property "Reference" "U4"
+		(property "Reference" "U5"
 			(at 167.64 240.03 0)
 			(effects
@@
 			)
 		)
-		(property "Value" "logic_nand"
+		(property "Value" "logic_and"
 			(at 151.13 234.95 0)
 			(effects
@@
 			)
 		)
+		(property "Campo4" "PUERTA NAND"
+			(at 174.625 240.03 0)
+			(effects
+				(font
+					(size 2.54 2.54)
+				)
+				(justify left)
+				(hide yes)
+			)
+		)
 		(pin ""
 		)
@@
 		)
 		(instances
-			(project "electric-simbolos-nombres"
+			(project ""
+				(path "/275d908d-d95f-4e76-9103-a82879596f4e"
+					(reference "U5")
+					(unit 1)
+				)
 				(path "/275d908d-d95f-4e76-9103-a82879596f4e/00000000-0000-0000-0000-00005bc9ce01"
-					(reference "U4")
+					(reference "U5")
 					(unit 1)
 				)
@@
 		(on_board yes)
 		(dnp no)
-		(property "Reference" "U2"
+		(property "Reference" "U3"
 			(at 167.64 209.55 0)
 			(effects
@@
 			)
 		)
-		(property "Value" "logic_or"
+		(property "Value" "logic_and"
 			(at 151.13 204.47 0)
 			(effects
@@
 			)
 		)
+		(property "Campo4" "PUERTA OR"
+			(at 174.625 209.55 0)
+			(effects
+				(font
+					(size 2.54 2.54)
+				)
+				(justify left)
+				(hide yes)
+			)
+		)
 		(pin ""
 		)
@@
 		)
 		(instances
-			(project "electric-simbolos-nombres"
+			(project ""
+				(path "/275d908d-d95f-4e76-9103-a82879596f4e"
+					(reference "U3")
+					(unit 1)
+				)
 				(path "/275d908d-d95f-4e76-9103-a82879596f4e/00000000-0000-0000-0000-00005bc9ce01"
-					(reference "U2")
+					(reference "U3")
 					(unit 1)
 				)

Commit message: 20/04/2026 Update
Parts:
- added M4: marco_1, symbol electric-simbolos-nombres-rescue:marco_1-simbolos
- added X1: ~, symbol simbolos-electricos:Borna
- CP3: License CC BY-SA 4.0 -> Licencia CC BY-SA 4.0
- renumbered C2 to C1, C1 to C2
