File: source/electric/electric-symbols-names/electric-names.kicad_sch (KiCad schematic)
At the start: 49 parts

Commit message: 20/04/2026 Update
Parts:
- added M3: marco_1, symbol electric-symbols-names-rescue:marco_1-simbolos
- CP2: License CC BY-SA 4.0 -> License CC BY-SA 4.0
Other:
- note added: "CONNECTION TERMINAL"
Changed lines of the file:
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@@
 (kicad_sch
-	(version 20231120)
+	(version 20250114)
 	(generator "eeschema")
-	(generator_version "8.0")
+	(generator_version "9.0")
 	(paper "A4" portrait)
 	(title_block
@@
 		(comment 2 "License CC BY-SA 4.0")
 	)
-	(polyline
-		(pts
-			(xy 205.74 292.1) (xy 205.74 7.62)
-		)
-		(stroke
-			(width 0)
-			(type default)
-		)
-	)
-	(polyline
-		(pts
-			(xy 5.08 7.62) (xy 205.74 7.62)
-		)
-		(stroke
-			(width 0)
-			(type default)
-		)
-	)
-	(polyline
-		(pts
-			(xy 5.08 292.1) (xy 5.08 7.62)
-		)
-		(stroke
-			(width 0)
-			(type default)
-		)
-	)
-	(polyline
-		(pts
-			(xy 5.08 292.1) (xy 205.74 292.1)
-		)
-		(stroke
-			(width 0)
-			(type default)
-		)
-	)
 	(text "BULB LAMP"
 		(exclude_from_sim no)
@@
 	(text "EARTH GROUND\nCONNECTOR"
 		(exclude_from_sim no)
-		(at 107.315 228.6 0)
+		(at 107.315 243.84 0)
 		(effects
 			(font
@@
 	(text "WIRES WITH\nCONNECTION"
 		(exclude_from_sim no)
-		(at 107.442 213.36 0)
+		(at 107.442 228.6 0)
 		(effects
 			(font
@@
 	(text "WIRES WITHOUT\nCONNECTION"
 		(exclude_from_sim no)
-		(at 107.442 198.12 0)
+		(at 107.442 213.36 0)
 		(effects
 			(font
@@
 		)
 	)
+	(text "CONNECTION\nTERMINAL"
+		(exclude_from_sim no)
+		(at 107.442 198.12 0)
+		(effects
+			(font
+				(size 2.54 2.54)
+			)
+			(justify left bottom)
+		)
+	)
 	(text "INDUCTOR/COIL"
 		(exclude_from_sim no)
@@
 	(text "CHASSIS\nGROUND\nCONNECTOR\n"
 		(exclude_from_sim no)
-		(at 107.315 245.745 0)
+		(at 107.315 260.985 0)
 		(effects
 			(font
@@
 		)
 	)
+	(polyline
+		(pts
+			(xy 205.74 292.1) (xy 205.74 7.62)
+		)
+		(stroke
+			(width 0)
+			(type default)
+		)
+	)
+	(polyline
+		(pts
+			(xy 5.08 7.62) (xy 205.74 7.62)
+		)
+		(stroke
+			(width 0)
+			(type default)
+		)
+	)
+	(polyline
+		(pts
+			(xy 5.08 292.1) (xy 5.08 7.62)
+		)
+		(stroke
+			(width 0)
+			(type default)
+		)
+	)
+	(polyline
+		(pts
+			(xy 5.08 292.1) (xy 205.74 292.1)
+		)
+		(stroke
+			(width 0)
+			(type default)
+		)
+	)
 	(symbol
 		(lib_id "electric-symbols-names-rescue:marco_2-simbolos")
@@
 	(symbol
 		(lib_id "electric-symbols-names-rescue:marco_1-simbolos")
-		(at 72.39 186.69 0)
+		(at 72.39 201.93 0)
 		(unit 1)
 		(exclude_from_sim no)
@@
 		(dnp no)
 		(property "Reference" "M?"
-			(at 75.565 191.135 0)
+			(at 75.565 206.375 0)
 			(effects
 				(font
@@
 		)
 		(property "Value" "marco_1"
-			(at 76.2 187.96 0)
+			(at 76.2 203.2 0)
 			(effects
 				(font
@@
 		)
 		(property "Footprint" ""
-			(at 73.66 190.5 0)
+			(at 73.66 205.74 0)
 			(effects
 				(font
@@
 		)
 		(property "Datasheet" ""
-			(at 73.66 190.5 0)
+			(at 73.66 205.74 0)
 			(effects
 				(font
@@
 		)
 		(property "Description" ""
-			(at 72.39 186.69 0)
+			(at 72.39 201.93 0)
 			(effects
 				(font
@@
 	(symbol
 		(lib_id "electric-symbols-names-rescue:marco_1-simbolos")
-		(at 72.39 201.93 0)
+		(at 72.39 217.17 0)
 		(unit 1)
 		(exclude_from_sim no)
@@
 		(dnp no)
 		(property "Reference" "M?"
-			(at 75.565 206.375 0)
+			(at 75.565 221.615 0)
 			(effects
 				(font
@@
 		)
 		(property "Value" "marco_1"
-			(at 76.2 203.2 0)
+			(at 76.2 218.44 0)
 			(effects
 				(font
@@
 		)
 		(property "Footprint" ""
-			(at 73.66 205.74 0)
+			(at 73.66 220.98 0)
 			(effects
 				(font
@@
 		)
 		(property "Datasheet" ""
-			(at 73.66 205.74 0)
+			(at 73.66 220.98 0)
 			(effects
 				(font
@@
 		)
 		(property "Description" ""
-			(at 72.39 201.93 0)
+			(at 72.39 217.17 0)
 			(effects
 				(font
@@
 	(symbol
 		(lib_id "electric-symbols-names-rescue:marco_1-simbolos")
-		(at 72.39 217.17 0)
+		(at 72.39 232.41 0)
 		(unit 1)
 		(exclude_from_sim no)
@@
 		(dnp no)
 		(property "Reference" "M?"
-			(at 75.565 221.615 0)
+			(at 75.565 236.855 0)
 			(effects
 				(font
@@
 		)
 		(property "Value" "marco_1"
-			(at 76.2 218.44 0)
+			(at 76.2 233.68 0)
 			(effects
 				(font
@@
 		)
 		(property "Footprint" ""
-			(at 73.66 220.98 0)
+			(at 73.66 236.22 0)
 			(effects
 				(font
@@
 		)
 		(property "Datasheet" ""
-			(at 73.66 220.98 0)
+			(at 73.66 236.22 0)
 			(effects
 				(font
@@
 		)
 		(property "Description" ""
-			(at 72.39 217.17 0)
+			(at 72.39 232.41 0)
 			(effects
 				(font
@@
 	(symbol
 		(lib_id "electric-symbols-names-rescue:marco_1-simbolos")
-		(at 72.39 232.41 0)
+		(at 72.39 247.65 0)
 		(unit 1)
 		(exclude_from_sim no)
@@
 		(dnp no)
 		(property "Reference" "M?"
-			(at 75.565 236.855 0)
+			(at 75.565 252.095 0)
 			(effects
 				(font
@@
 		)
 		(property "Value" "marco_1"
-			(at 76.2 233.68 0)
+			(at 76.2 248.92 0)
 			(effects
 				(font
@@
 		)
 		(property "Footprint" ""
-			(at 73.66 236.22 0)
+			(at 73.66 251.46 0)
 			(effects
 				(font
@@
 		)
 		(property "Datasheet" ""
-			(at 73.66 236.22 0)
+			(at 73.66 251.46 0)
 			(effects
 				(font
@@
 		)
 		(property "Description" ""
-			(at 72.39 232.41 0)
+			(at 72.39 247.65 0)
 			(effects
 				(font
@@
 	)
 	(symbol
+		(lib_id "electric-symbols-names-rescue:marco_1-simbolos")
+		(at 72.39 186.69 0)
+		(unit 1)
+		(exclude_from_sim no)
+		(in_bom yes)
+		(on_board yes)
+		(dnp no)
+		(property "Reference" "M3"
+			(at 75.565 191.135 0)
+			(effects
+				(font
+					(size 2.54 2.54)
+				)
+				(hide yes)
+			)
+		)
+		(property "Value" "marco_1"
+			(at 76.2 187.96 0)
+			(effects
+				(font
+					(size 1.27 1.27)
+				)
+				(hide yes)
+			)
+		)
+		(property "Footprint" ""
+			(at 73.66 190.5 0)
+			(effects
+				(font
+					(size 1.27 1.27)
+				)
+				(hide yes)
+			)
+		)
+		(property "Datasheet" ""
+			(at 73.66 190.5 0)
+			(effects
+				(font
+					(size 1.27 1.27)
+				)
+				(hide yes)
+			)
+		)
+		(property "Description" ""
+			(at 72.39 186.69 0)
+			(effects
+				(font
+					(size 1.27 1.27)
+				)
+				(hide yes)
+			)
+		)
+		(instances
+			(project "electric-symbols-names"
+				(path "/275d908d-d95f-4e76-9103-a82879596f4e/00000000-0000-0000-0000-00005bc9cadf"
+					(reference "M3")
+					(unit 1)
+				)
+			)
+		)
+	)
+	(symbol
 		(lib_id "simbolos-electricos:CopyRight")
 		(at 101.6 292.1 0)
@@
 			)
 		)
-		(property "License" "CC BY-SA 4.0"
-			(at 101.6 287.02 0)
+		(property "License" "License CC BY-SA 4.0"
+			(at 101.6 285.75 0)
 			(effects
 				(font
-					(size 1.778 1.778)
+					(size 1.905 1.905)
 				)
 			)
@@
 			(effects
 				(font
-					(size 1.778 1.778)
+					(size 1.905 1.905)
 				)
 			)
