File: source/electric/electric-symbols-names/electric-symbols-names.kicad_sch (KiCad schematic)
At the start: 88 parts, among them J1 conector, K1 CONTACTO, K1 RELE, M1 MOTOR, Q1 TRANSISTOR, Q2 TRANSISTOR, U1 OA, U1 logic_and, U2 logic_and, U3 logic_and, U4 logic_and, U5 logic_and, U6 logic_and

Commit message: 18/03/2025 Update
Changed lines of the file:
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@@
-	)
-	(symbol
-		(lib_id "simbolos-electricos:resistencia_2")
-		(at 11.43 137.16 90)
-		(mirror x)
-		(unit 1)
-		(exclude_from_sim no)
-		(in_bom yes)
-		(on_board yes)
-		(dnp no)
-		(property "Reference" "R5"
-			(at 16.51 142.24 90)
-			(effects
-				(font
-					(size 2.54 2.54)
-				)
-				(hide yes)
-			)
-		)
-		(property "Value" "resistencia"
-			(at 17.145 134.62 90)
-			(effects
-				(font
-					(size 1.27 1.27)
-				)
-				(hide yes)
-			)
-		)
-		(property "Footprint" ""
-			(at 13.97 139.7 0)
-			(effects
-				(font
-					(size 1.27 1.27)
-				)
-				(hide yes)
-			)
-		)
-		(property "Datasheet" ""
-			(at 13.97 139.7 0)
-			(effects
-				(font
-					(size 1.27 1.27)
-				)
-				(hide yes)
-			)
-		)
-		(property "Description" ""
-			(at 11.43 137.16 0)
-			(effects
-				(font
-					(size 1.27 1.27)
-				)
-				(hide yes)
-			)
-		)
-		(pin ""
-		)
-		(pin ""
-		)
-		(instances
-			(project ""
-				(path "/275d908d-d95f-4e76-9103-a82879596f4e"
-					(reference "R5")
-					(unit 1)
-				)
-			)
-		)
 	)
 	(symbol
@@
 					(unit 1)
 				)
+			)
+		)
+	)
+	(symbol
+		(lib_id "simbolos-electricos:resistencia_2")
+		(at 11.43 137.16 90)
+		(unit 1)
+		(exclude_from_sim no)
+		(in_bom yes)
+		(on_board yes)
+		(dnp no)
+		(fields_autoplaced yes)
+		(property "Reference" "R5"
+			(at 16.51 132.08 90)
+			(effects
+				(font
+					(size 2.54 2.54)
+				)
+				(hide yes)
+			)
+		)
+		(property "Value" "resistencia"
+			(at 17.145 139.7 90)
+			(effects
+				(font
+					(size 1.27 1.27)
+				)
+				(hide yes)
+			)
+		)
+		(property "Footprint" ""
+			(at 13.97 134.62 0)
+			(effects
+				(font
+					(size 1.27 1.27)
+				)
+				(hide yes)
+			)
+		)
+		(property "Datasheet" ""
+			(at 13.97 134.62 0)
+			(effects
+				(font
+					(size 1.27 1.27)
+				)
+				(hide yes)
+			)
+		)
+		(property "Description" ""
+			(at 11.43 137.16 0)
+			(effects
+				(font
+					(size 1.27 1.27)
+				)
+				(hide yes)
+			)
+		)
+		(pin ""
+		)
+		(pin ""
+		)
+		(instances
+			(project ""
+				(path "/275d908d-d95f-4e76-9103-a82879596f4e"
+					(reference "R5")
+					(unit 1)
+				)

Commit message: 28/07/2025 Update
Parts:
- renumbered U1 to U2, U2 to U3, U3 to U4, U4 to U5, U5 to U6, U6 to U7
Changed lines of the file:
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@@
 		(on_board yes)
 		(dnp no)
-		(property "Reference" "U1"
+		(property "Reference" "U2"
 			(at 167.64 194.31 0)
 			(effects
@@
 			(project "electric-symbols-names"
 				(path "/275d908d-d95f-4e76-9103-a82879596f4e"
-					(reference "U1")
+					(reference "U2")
 					(unit 1)
 				)
@@
 		(on_board yes)
 		(dnp no)
-		(property "Reference" "U2"
+		(property "Reference" "U3"
 			(at 167.64 209.55 0)
 			(effects
@@
 			(project "electric-symbols-names"
 				(path "/275d908d-d95f-4e76-9103-a82879596f4e"
-					(reference "U2")
+					(reference "U3")
 					(unit 1)
 				)
@@
 		(on_board yes)
 		(dnp no)
-		(property "Reference" "U3"
+		(property "Reference" "U4"
 			(at 167.64 224.79 0)
 			(effects
@@
 			(project "electric-symbols-names"
 				(path "/275d908d-d95f-4e76-9103-a82879596f4e"
-					(reference "U3")
+					(reference "U4")
 					(unit 1)
 				)
@@
 		(on_board yes)
 		(dnp no)
-		(property "Reference" "U4"
+		(property "Reference" "U5"
 			(at 167.64 240.03 0)
 			(effects
@@
 			(project "electric-symbols-names"
 				(path "/275d908d-d95f-4e76-9103-a82879596f4e"
-					(reference "U4")
+					(reference "U5")
 					(unit 1)
 				)
@@
 		(on_board yes)
 		(dnp no)
-		(property "Reference" "U5"
+		(property "Reference" "U6"
 			(at 167.64 255.27 0)
 			(effects
@@
 			(project "electric-symbols-names"
 				(path "/275d908d-d95f-4e76-9103-a82879596f4e"
-					(reference "U5")
+					(reference "U6")
 					(unit 1)
 				)
@@
 		(on_board yes)
 		(dnp no)
-		(property "Reference" "U6"
+		(property "Reference" "U7"
 			(at 167.64 270.51 0)
 			(effects
@@
 			(project "electric-symbols-names"
 				(path "/275d908d-d95f-4e76-9103-a82879596f4e"
-					(reference "U6")
+					(reference "U7")
 					(unit 1)
 				)
@@
 		)
 		(instances
-			(project "electric-symbols-names"
+			(project ""
 				(path "/275d908d-d95f-4e76-9103-a82879596f4e"
 					(reference "U1")

Commit message: 20/04/2026 Update
Parts:
- added M2: marco_1, symbol electric-symbols-names-rescue:marco_1-simbolos
- added X1: ~, symbol simbolos-electricos:Borna
- CP1: License CC BY-SA 4.0 -> License CC BY-SA 4.0
Other:
- note added: "CONNECTION TERMINAL"
