File: source/electric/electric-symbols-names/electric-symbols.kicad_sch (KiCad schematic)
At the start: 87 parts, among them J1 conector, K1 CONTACTO, K1 RELE, M1 MOTOR, Q1 TRANSISTOR, Q2 TRANSISTOR, U1 OA, U1 logic_and, U2 logic_and, U3 logic_and, U4 logic_and, U5 logic_and, U6 logic_and

Commit message: 17/03/2025 Update
Parts:
- added R6: resistencia, symbol simbolos-electricos:resistencia_2
- V? (x2): value CONEXIÓN -> CONNECTION
Other:
- moved on the sheet: R1

Commit message: 18/03/2025 Update
Parts:
- removed R6: resistencia, symbol simbolos-electricos:resistencia_2
- added R1: resistencia, symbol simbolos-electricos:resistencia_2
Changed lines of the file:
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@@
-	)
-	(symbol
-		(lib_id "simbolos-electricos:resistencia_2")
-		(at 11.43 137.16 90)
-		(unit 1)
-		(exclude_from_sim no)
-		(in_bom yes)
-		(on_board yes)
-		(dnp no)
-		(fields_autoplaced yes)
-		(property "Reference" "R6"
-			(at 16.51 132.08 90)
-			(effects
-				(font
-					(size 2.54 2.54)
-				)
-				(hide yes)
-			)
-		)
-		(property "Value" "resistencia"
-			(at 17.145 139.7 90)
-			(effects
-				(font
-					(size 1.27 1.27)
-				)
-				(hide yes)
-			)
-		)
-		(property "Footprint" ""
-			(at 13.97 134.62 0)
-			(effects
-				(font
-					(size 1.27 1.27)
-				)
-				(hide yes)
-			)
-		)
-		(property "Datasheet" ""
-			(at 13.97 134.62 0)
-			(effects
-				(font
-					(size 1.27 1.27)
-				)
-				(hide yes)
-			)
-		)
-		(property "Description" ""
-			(at 11.43 137.16 0)
-			(effects
-				(font
-					(size 1.27 1.27)
-				)
-				(hide yes)
-			)
-		)
-		(pin ""
-		)
-		(pin ""
-		)
-		(instances
-			(project ""
-				(path "/275d908d-d95f-4e76-9103-a82879596f4e/00000000-0000-0000-0000-00005bc9ce01"
-					(reference "R6")
-					(unit 1)
-				)
-			)
-		)
 	)
 	(symbol
@@
 					(unit 1)
 				)
+			)
+		)
+	)
+	(symbol
+		(lib_id "simbolos-electricos:resistencia_2")
+		(at 11.43 137.16 90)
+		(unit 1)
+		(exclude_from_sim no)
+		(in_bom yes)
+		(on_board yes)
+		(dnp no)
+		(fields_autoplaced yes)
+		(property "Reference" "R1"
+			(at 16.51 132.08 90)
+			(effects
+				(font
+					(size 2.54 2.54)
+				)
+				(hide yes)
+			)
+		)
+		(property "Value" "resistencia"
+			(at 17.145 139.7 90)
+			(effects
+				(font
+					(size 1.27 1.27)
+				)
+				(hide yes)
+			)
+		)
+		(property "Footprint" ""
+			(at 13.97 134.62 0)
+			(effects
+				(font
+					(size 1.27 1.27)
+				)
+				(hide yes)
+			)
+		)
+		(property "Datasheet" ""
+			(at 13.97 134.62 0)
+			(effects
+				(font
+					(size 1.27 1.27)
+				)
+				(hide yes)
+			)
+		)
+		(property "Description" ""
+			(at 11.43 137.16 0)
+			(effects
+				(font
+					(size 1.27 1.27)
+				)
+				(hide yes)
+			)
+		)
+		(pin ""
+		)
+		(pin ""
+		)
+		(instances
+			(project ""
+				(path "/275d908d-d95f-4e76-9103-a82879596f4e/00000000-0000-0000-0000-00005bc9ce01"
+					(reference "R1")
+					(unit 1)
+				)

Commit message: 28/07/2025 Update
Changed lines of the file:
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@@
 		)
 		(instances
-			(project "electric-symbols-names"
-				(path "/275d908d-d95f-4e76-9103-a82879596f4e/00000000-0000-0000-0000-00005bc9ce01"
+			(project ""
+				(path "/275d908d-d95f-4e76-9103-a82879596f4e"
 					(reference "U1")
 					(unit 1)
 				)
+				(path "/275d908d-d95f-4e76-9103-a82879596f4e/00000000-0000-0000-0000-00005bc9ce01"
+					(reference "U2")
+					(unit 1)
+				)
 			)
 		)
@@
 		)
 		(instances
-			(project "electric-symbols-names"
-				(path "/275d908d-d95f-4e76-9103-a82879596f4e/00000000-0000-0000-0000-00005bc9ce01"
+			(project ""
+				(path "/275d908d-d95f-4e76-9103-a82879596f4e"
 					(reference "U2")
 					(unit 1)
 				)
+				(path "/275d908d-d95f-4e76-9103-a82879596f4e/00000000-0000-0000-0000-00005bc9ce01"
+					(reference "U3")
+					(unit 1)
+				)
 			)
 		)
@@
 		)
 		(instances
-			(project "electric-symbols-names"
-				(path "/275d908d-d95f-4e76-9103-a82879596f4e/00000000-0000-0000-0000-00005bc9ce01"
+			(project ""
+				(path "/275d908d-d95f-4e76-9103-a82879596f4e"
 					(reference "U3")
 					(unit 1)
 				)
+				(path "/275d908d-d95f-4e76-9103-a82879596f4e/00000000-0000-0000-0000-00005bc9ce01"
+					(reference "U4")
+					(unit 1)
+				)
 			)
 		)
@@
 		)
 		(instances
-			(project "electric-symbols-names"
-				(path "/275d908d-d95f-4e76-9103-a82879596f4e/00000000-0000-0000-0000-00005bc9ce01"
+			(project ""
+				(path "/275d908d-d95f-4e76-9103-a82879596f4e"
 					(reference "U4")
 					(unit 1)
 				)
+				(path "/275d908d-d95f-4e76-9103-a82879596f4e/00000000-0000-0000-0000-00005bc9ce01"
+					(reference "U5")
+					(unit 1)
+				)
 			)
 		)
@@
 		)
 		(instances
-			(project "electric-symbols-names"
-				(path "/275d908d-d95f-4e76-9103-a82879596f4e/00000000-0000-0000-0000-00005bc9ce01"
+			(project ""
+				(path "/275d908d-d95f-4e76-9103-a82879596f4e"
 					(reference "U5")
 					(unit 1)
 				)
+				(path "/275d908d-d95f-4e76-9103-a82879596f4e/00000000-0000-0000-0000-00005bc9ce01"
+					(reference "U6")
+					(unit 1)
+				)
 			)
 		)
@@
 		)
 		(instances
-			(project "electric-symbols-names"
-				(path "/275d908d-d95f-4e76-9103-a82879596f4e/00000000-0000-0000-0000-00005bc9ce01"
+			(project ""
+				(path "/275d908d-d95f-4e76-9103-a82879596f4e"
 					(reference "U6")
 					(unit 1)
 				)
+				(path "/275d908d-d95f-4e76-9103-a82879596f4e/00000000-0000-0000-0000-00005bc9ce01"
+					(reference "U7")
+					(unit 1)
+				)
 			)
 		)
@@
 	)
 	(symbol
-		(lib_id "simbolos-electricos:potenciometro")
-		(at 151.13 113.03 0)
+		(lib_id "simbolos-electricos:OA")
+		(at 146.685 87.63 0)
 		(unit 1)
 		(exclude_from_sim no)
@@
 		(on_board yes)
 		(dnp no)
-		(property "Reference" "R2"
-			(at 167.64 118.11 0)
+		(property "Reference" "U1"
+			(at 167.64 87.63 0)
 			(effects
 				(font
@@
 			)
 		)
-		(property "Value" "potenciometro"
-			(at 148.59 118.745 90)
+		(property "Value" "OA"
+			(at 153.035 83.82 0)
 			(effects
 				(font
@@
 		)
 		(property "Footprint" ""
-			(at 152.4 115.57 0)
+			(at 146.685 87.63 0)
 			(effects
 				(font
@@
 		)
 		(property "Datasheet" ""
-			(at 152.4 115.57 0)
+			(at 146.685 87.63 0)
 			(effects
 				(font
@@
 		)
 		(property "Description" ""
-			(at 151.13 113.03 0)
+			(at 146.685 87.63 0)
 			(effects
 				(font
@@
 		)
 		(instances
-			(project "electric-symbols-names"
+			(project ""
+				(path "/275d908d-d95f-4e76-9103-a82879596f4e"
+					(reference "U1")
+					(unit 1)
+				)
 				(path "/275d908d-d95f-4e76-9103-a82879596f4e/00000000-0000-0000-0000-00005bc9ce01"
-					(reference "R2")
+					(reference "U1")
 					(unit 1)
 				)
@@
 	)
 	(symbol
-		(lib_id "simbolos-electricos:CopyRight")
-		(at 101.6 292.1 0)
+		(lib_id "simbolos-electricos:potenciometro")
+		(at 151.13 113.03 0)
 		(unit 1)
 		(exclude_from_sim no)
@@
 		(on_board yes)
 		(dnp no)
-		(fields_autoplaced yes)
-		(property "Reference" "CP3"
-			(at 107.95 290.83 0)
+		(property "Reference" "R2"
+			(at 167.64 118.11 0)
 			(effects
 				(font
-					(size 1.016 1.016)
+					(size 2.54 2.54)
 				)
-				(hide yes)
 			)
 		)
-		(property "Value" "CopyRight"
-			(at 101.6 290.83 0)
+		(property "Value" "potenciometro"
+			(at 148.59 118.745 90)
 			(effects
 				(font
-					(size 1.016 1.016)
+					(size 1.27 1.27)
 				)
 				(hide yes)
@@
 		)
 		(property "Footprint" ""
-			(at 99.06 283.21 0)
+			(at 152.4 115.57 0)
 			(effects
 				(font
@@
 		)
 		(property "Datasheet" ""
-			(at 101.6 287.02 0)
+			(at 152.4 115.57 0)
 			(effects
 				(font
@@
 		)
 		(property "Description" ""
-			(at 101.6 292.1 0)
+			(at 151.13 113.03 0)
 			(effects
 				(font
@@
 			)
 		)
-		(property "License" "CC BY-SA 4.0"
-			(at 101.6 287.02 0)
-			(effects
-				(font
-					(size 1.778 1.778)
-				)
-			)
+		(pin ""
 		)
-		(property "Web" "www.picuino.com"
-			(at 101.6 289.56 0)
-			(effects
-				(font
-					(size 1.778 1.778)
-				)
-			)
+		(pin ""
+		)
+		(pin ""
 		)
 		(instances
 			(project "electric-symbols-names"
 				(path "/275d908d-d95f-4e76-9103-a82879596f4e/00000000-0000-0000-0000-00005bc9ce01"
-					(reference "CP3")
+					(reference "R2")
 					(unit 1)
 				)
@@
 	)
 	(symbol
-		(lib_id "simbolos-electricos:resistencia_2")
-		(at 11.43 137.16 90)
+		(lib_id "simbolos-electricos:CopyRight")
+		(at 101.6 292.1 0)
 		(unit 1)
 		(exclude_from_sim no)
@@
 		(dnp no)
 		(fields_autoplaced yes)
-		(property "Reference" "R1"
-			(at 16.51 132.08 90)
+		(property "Reference" "CP3"
+			(at 107.95 290.83 0)
 			(effects
 				(font
-					(size 2.54 2.54)
+					(size 1.016 1.016)
 				)
 				(hide yes)
 			)
 		)
-		(property "Value" "resistencia"
-			(at 17.145 139.7 90)
+		(property "Value" "CopyRight"
+			(at 101.6 290.83 0)
 			(effects
 				(font
-					(size 1.27 1.27)
+					(size 1.016 1.016)
 				)
 				(hide yes)
@@
 		)
 		(property "Footprint" ""
-			(at 13.97 134.62 0)
+			(at 99.06 283.21 0)
 			(effects
 				(font
@@
 		)
 		(property "Datasheet" ""
-			(at 13.97 134.62 0)
+			(at 101.6 287.02 0)
 			(effects
 				(font
@@
 		)
 		(property "Description" ""
-			(at 11.43 137.16 0)
+			(at 101.6 292.1 0)
 			(effects
 				(font
@@
 			)
 		)
-		(pin ""
+		(property "License" "CC BY-SA 4.0"
+			(at 101.6 287.02 0)
+			(effects
+				(font
+					(size 1.778 1.778)
+				)
+			)
 		)
-		(pin ""
+		(property "Web" "www.picuino.com"
+			(at 101.6 289.56 0)
+			(effects
+				(font
+					(size 1.778 1.778)
+				)
+			)
 		)
 		(instances
-			(project ""
+			(project "electric-symbols-names"
 				(path "/275d908d-d95f-4e76-9103-a82879596f4e/00000000-0000-0000-0000-00005bc9ce01"
-					(reference "R1")
+					(reference "CP3")
 					(unit 1)
 				)
@@
 	)
 	(symbol
-		(lib_id "simbolos-electricos:OA")
-		(at 146.685 87.63 0)
+		(lib_id "simbolos-electricos:resistencia_2")
+		(at 11.43 137.16 90)
 		(unit 1)
 		(exclude_from_sim no)
@@
 		(on_board yes)
 		(dnp no)
-		(property "Reference" "U1"
-			(at 167.64 87.63 0)
+		(fields_autoplaced yes)
+		(property "Reference" "R1"
+			(at 16.51 132.08 90)
 			(effects
 				(font
 					(size 2.54 2.54)
 				)
+				(hide yes)
 			)
 		)
-		(property "Value" "OA"
-			(at 153.035 83.82 0)
+		(property "Value" "resistencia"
+			(at 17.145 139.7 90)
 			(effects
 				(font
@@
 		)
 		(property "Footprint" ""
-			(at 146.685 87.63 0)
+			(at 13.97 134.62 0)
 			(effects
 				(font
@@
 		)
 		(property "Datasheet" ""
-			(at 146.685 87.63 0)
+			(at 13.97 134.62 0)
 			(effects
 				(font
@@
 		)
 		(property "Description" ""
-			(at 146.685 87.63 0)
+			(at 11.43 137.16 0)
 			(effects
 				(font
@@
 		(pin ""
 		)
-		(pin ""
-		)
 		(instances
-			(project "electric-symbols-names"
+			(project ""
 				(path "/275d908d-d95f-4e76-9103-a82879596f4e/00000000-0000-0000-0000-00005bc9ce01"
-					(reference "U1")
+					(reference "R1")
 					(unit 1)
 				)

Commit message: 20/04/2026 Update
Parts:
- added M4: marco_1, symbol electric-symbols-names-rescue:marco_1-simbolos
- added X1: ~, symbol simbolos-electricos:Borna
- CP3: License CC BY-SA 4.0 -> License CC BY-SA 4.0
- renumbered U1 to U2, U2 to U3, U3 to U4, U4 to U5, U5 to U6, U6 to U7
