File: source/cucabot/cucabot-cero-electric/cucabot-cero-electric.kicad_sch (KiCad schematic)
At the start: 20 parts, among them M1 motor, M2 motor, X1-X6 borna_6x2

Commit message: 21/04/2026 Update
Connections:
- net at V2., X1-X6.: no longer V1.
- net at S1.: now also X1-X6.
- net at S2.: now also X1.; no longer X3.
- new net: V1., V2., X1-X6.
- new net: V1., V2., X2.
- new net: S1., X1-X6.
- new net: S2., X3.
- new net: S2., X5., X6.
- new net: M1., M2., X4.
- new net: M1. (V-), M2. (V-), X1-X6.
- new net: S2., X1-X6. (x2)
Other:
- note added: "SENSOR DEL PARACHOQUES"
- note removed: "ANTENA FRONTAL"
- moved on the sheet: V1, V2
Changed lines of the file:
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@@
 		)
 	)
-	(text "ANTENA FRONTAL"
+	(text "SENSOR DEL\nPARACHOQUES"
 		(exclude_from_sim no)
 		(at 145.288 63.5 0)
@@
 	(wire
 		(pts
-			(xy 44.45 69.85) (xy 44.45 66.04)
+			(xy 44.45 72.39) (xy 44.45 66.04)
 		)
 		(stroke
@@
 	(wire
 		(pts
-			(xy 44.45 49.53) (xy 44.45 39.37)
+			(xy 44.45 46.99) (xy 44.45 39.37)
 		)
 		(stroke
@@
 	(polyline
 		(pts
-			(xy 87.63 50.8) (xy 87.63 51.435)
+			(xy 97.79 50.8) (xy 97.79 51.435)
 		)
 		(stroke
@@
 	(polyline
 		(pts
-			(xy 87.63 69.215) (xy 87.63 71.12)
+			(xy 97.79 69.215) (xy 97.79 71.12)
 		)
 		(stroke
@@
 	(wire
 		(pts
-			(xy 44.45 60.96) (xy 44.45 57.15)
+			(xy 44.45 60.96) (xy 44.45 54.61)
 		)
 		(stroke
@@
 	(polyline
 		(pts
-			(xy 86.36 70.485) (xy 88.9 70.485)
+			(xy 96.52 70.485) (xy 99.06 70.485)
 		)
 		(stroke
@@
 	(wire
 		(pts
-			(xy 44.45 77.47) (xy 44.45 88.9)
+			(xy 44.45 80.01) (xy 44.45 88.9)
 		)
 		(stroke
@@
 	(polyline
 		(pts
-			(xy 87.63 48.895) (xy 87.63 50.8)
+			(xy 97.79 48.895) (xy 97.79 50.8)
 		)
 		(stroke
@@
 	(polyline
 		(pts
-			(xy 86.36 50.165) (xy 88.9 50.165)
+			(xy 96.52 50.165) (xy 99.06 50.165)
 		)
 		(stroke
@@
 	(polyline
 		(pts
-			(xy 87.63 71.12) (xy 87.63 71.755)
+			(xy 97.79 71.12) (xy 97.79 71.755)
 		)
 		(stroke
@@
 	(symbol
 		(lib_id "simbolos:Pila")
-		(at 44.45 49.53 0)
+		(at 44.45 46.99 0)
 		(unit 1)
 		(exclude_from_sim no)
@@
 		(dnp no)
 		(property "Reference" "V1"
-			(at 49.0982 53.34 0)
+			(at 49.0982 50.8 0)
 			(effects
 				(font
@@
 		)
 		(property "Value" "Pila"
-			(at 46.99 51.435 0)
+			(at 46.99 48.895 0)
 			(effects
 				(font
@@
 		)
 		(property "Footprint" ""
-			(at 44.45 52.705 0)
+			(at 44.45 50.165 0)
 			(effects
 				(font
@@
 		)
 		(property "Datasheet" ""
-			(at 44.45 52.705 0)
+			(at 44.45 50.165 0)
 			(effects
 				(font
@@
 		)
 		(property "Description" ""
-			(at 44.45 49.53 0)
+			(at 44.45 46.99 0)
 			(effects
 				(font
@@
 		)
 		(instances
-			(project "cucabot-cero"
+			(project "cucabot-cero-electric"
 				(path "/91e6286f-2f5f-4c12-b8bc-a46dfa772353"
 					(reference "M2")
@@
 		)
 		(instances
-			(project "cucabot-cero"
+			(project "cucabot-cero-electric"
 				(path "/91e6286f-2f5f-4c12-b8bc-a46dfa772353"
 					(reference "X2")
@@
 		(lib_name "Motor_DC_1")
 		(lib_id "electric-simbolos:Motor_DC")
-		(at 39.37 227.33 0)
+		(at 39.37 234.95 0)
+		(mirror x)
 		(unit 1)
 		(exclude_from_sim no)
@@
 		(dnp no)
 		(property "Reference" "M1"
-			(at 24.638 231.394 0)
+			(at 24.638 230.886 0)
 			(effects
 				(font
@@
 		)
 		(property "Value" "~"
-			(at 39.37 224.79 0)
+			(at 39.37 237.49 0)
 			(effects
 				(font
@@
 		)
 		(property "Footprint" ""
-			(at 39.37 227.33 0)
+			(at 39.37 234.95 0)
 			(effects
 				(font
@@
 		)
 		(property "Datasheet" ""
-			(at 39.37 227.33 0)
+			(at 39.37 234.95 0)
 			(effects
 				(font
@@
 		)
 		(property "Description" ""
-			(at 39.37 227.33 0)
+			(at 39.37 234.95 0)
 			(effects
 				(font
@@
 		(lib_name "Pila_1")
 		(lib_id "simbolos:Pila")
-		(at 44.45 69.85 0)
+		(at 44.45 72.39 0)
 		(unit 1)
 		(exclude_from_sim no)
@@
 		(dnp no)
 		(property "Reference" "V2"
-			(at 49.0982 73.66 0)
+			(at 49.0982 76.2 0)
 			(effects
 				(font
@@
 		)
 		(property "Value" "Pila"
-			(at 46.99 71.755 0)
+			(at 46.99 74.295 0)
 			(effects
 				(font
@@
 		)
 		(property "Footprint" ""
-			(at 44.45 73.025 0)
+			(at 44.45 75.565 0)
 			(effects
 				(font
@@
 		)
 		(property "Datasheet" ""
-			(at 44.45 73.025 0)
+			(at 44.45 75.565 0)
 			(effects
 				(font
@@
 		)
 		(property "Description" ""
-			(at 44.45 69.85 0)
+			(at 44.45 72.39 0)
 			(effects
 				(font
@@
 		)
 		(instances
-			(project "cucabot-cero"
+			(project "cucabot-cero-electric"
 				(path "/91e6286f-2f5f-4c12-b8bc-a46dfa772353"
 					(reference "V2")
@@
 		(lib_name "Motor_DC_2")
 		(lib_id "electric-simbolos:Motor_DC")
-		(at 39.37 240.03 0)
+		(at 39.37 247.65 0)
+		(mirror x)
 		(unit 1)
 		(exclude_from_sim no)
@@
 		(dnp no)
 		(property "Reference" "M2"
-			(at 24.638 244.094 0)
+			(at 24.638 243.586 0)
 			(effects
 				(font
@@
 		)
 		(property "Value" "~"
-			(at 39.37 237.49 0)
+			(at 39.37 250.19 0)
 			(effects
 				(font
@@
 		)
 		(property "Footprint" ""
-			(at 39.37 240.03 0)
+			(at 39.37 247.65 0)
 			(effects
 				(font
@@
 		)
 		(property "Datasheet" ""
-			(at 39.37 240.03 0)
+			(at 39.37 247.65 0)
 			(effects
 				(font
@@
 		)
 		(property "Description" ""
-			(at 39.37 240.03 0)
+			(at 39.37 247.65 0)
 			(effects
 				(font
@@
 		)
 		(instances
-			(project "cucabot-cero"
+			(project "cucabot-cero-electric"
 				(path "/91e6286f-2f5f-4c12-b8bc-a46dfa772353"
 					(reference "M2")
@@
 		)
 		(instances
-			(project "cucabot-cero"
+			(project "cucabot-cero-electric"
 				(path "/91e6286f-2f5f-4c12-b8bc-a46dfa772353"
 					(reference "M1")
@@
 		)
 		(instances
-			(project "cucabot-cero"
+			(project "cucabot-cero-electric"
 				(path "/91e6286f-2f5f-4c12-b8bc-a46dfa772353"
 					(reference "X4")
@@
 		)
 		(instances
-			(project "cucabot-cero"
+			(project "cucabot-cero-electric"
 				(path "/91e6286f-2f5f-4c12-b8bc-a46dfa772353"
 					(reference "X5")
@@
 		)
 		(instances
-			(project "cucabot-cero"
+			(project "cucabot-cero-electric"
 				(path "/91e6286f-2f5f-4c12-b8bc-a46dfa772353"
 					(reference "X6")
@@
 		)
 		(instances
-			(project "cucabot-cero"
+			(project "cucabot-cero-electric"
 				(path "/91e6286f-2f5f-4c12-b8bc-a46dfa772353"
 					(reference "V2")
@@
 		)
 		(instances
-			(project "cucabot-cero"
+			(project "cucabot-cero-electric"
 				(path "/91e6286f-2f5f-4c12-b8bc-a46dfa772353"
 					(reference "X1")
