File: source/cucabot/cucabot-cero-electric/cucabot-cero-electric.kicad_sch (KiCad schematic)
At the start: 20 parts, among them M1 motor, M2 motor, X1 borna_6x2

Commit message: 27/04/2026 Update
Connections:
- net at V2., X1.: no longer V1.
- net at S1.: now also X1.
- net at X2.: now also V1., V2.; no longer S1.
- net at S2.: now also X1.; no longer X3.
- new net: V1., V2., X1.
- new net: S1., X1.
- new net: M1., M2., X4.
- new net: S1., X2.
- new net: S2., X3.
- new net: M1. (-), M2. (-), X1.
- new net: S2., X1. (x2)
Other:
- note added: "ROBOT CUCABOT CERO"
- note added: "SELECTOR DE MARCHA"
- note removed: "ROBOT CUCABOT MURÓFILO"
Changed lines of the file:
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@@
+		)
+	)
+	(text "SELECTOR\nDE MARCHA"
+		(exclude_from_sim no)
+		(at 147.574 63.5 0)
+		(effects
+			(font
+				(size 1.905 1.905)
+			)
+			(justify left)
 		)
 	)
@@
 		)
 	)
-	(text "ROBOT CUCABOT MURÓFILO"
+	(text "ROBOT CUCABOT CERO"
 		(exclude_from_sim no)
 		(at 105.41 12.7 0)
@@
 	)
 	(symbol
+		(lib_id "electric-simbolos:selector")
+		(at 129.54 63.5 0)
+		(unit 1)
+		(exclude_from_sim no)
+		(in_bom yes)
+		(on_board yes)
+		(dnp no)
+		(property "Reference" "S2"
+			(at 133.35 57.658 0)
+			(effects
+				(font
+					(size 2.54 2.54)
+				)
+			)
+		)
+		(property "Value" "selector"
+			(at 129.54 64.77 0)
+			(effects
+				(font
+					(size 1.27 1.27)
+				)
+				(hide yes)
+			)
+		)
+		(property "Footprint" ""
+			(at 137.16 67.31 0)
+			(effects
+				(font
+					(size 1.27 1.27)
+				)
+				(hide yes)
+			)
+		)
+		(property "Datasheet" ""
+			(at 137.16 67.31 0)
+			(effects
+				(font
+					(size 1.27 1.27)
+				)
+				(hide yes)
+			)
+		)
+		(property "Description" ""
+			(at 129.54 63.5 0)
+			(effects
+				(font
+					(size 1.27 1.27)
+				)
+				(hide yes)
+			)
+		)
+		(pin ""
+		)
+		(pin ""
+		)
+		(pin ""
+		)
+		(instances
+			(project ""
+				(path "/91e6286f-2f5f-4c12-b8bc-a46dfa772353"
+					(reference "S2")
+					(unit 1)
+				)
+			)
+		)
+	)
+	(symbol
 		(lib_name "Motor_DC_2")
 		(lib_id "electric-simbolos:Motor_DC")
@@
 					(unit 1)
 				)
-			)
-		)
-	)
-	(symbol
-		(lib_id "electric-simbolos:selector")
-		(at 129.54 63.5 0)
-		(unit 1)
-		(exclude_from_sim no)
-		(in_bom yes)
-		(on_board yes)
-		(dnp no)
-		(fields_autoplaced yes)
-		(property "Reference" "S2"
-			(at 135.89 55.88 0)
-			(effects
-				(font
-					(size 2.54 2.54)
-				)
-			)
-		)
-		(property "Value" "selector"
-			(at 129.54 64.77 0)
-			(effects
-				(font
-					(size 1.27 1.27)
-				)
-				(hide yes)
-			)
-		)
-		(property "Footprint" ""
-			(at 137.16 67.31 0)
-			(effects
-				(font
-					(size 1.27 1.27)
-				)
-				(hide yes)
-			)
-		)
-		(property "Datasheet" ""
-			(at 137.16 67.31 0)
-			(effects
-				(font
-					(size 1.27 1.27)
-				)
-				(hide yes)
-			)
-		)
-		(property "Description" ""
-			(at 129.54 63.5 0)
-			(effects
-				(font
-					(size 1.27 1.27)
-				)
-				(hide yes)
-			)
-		)
-		(pin ""
-		)
-		(pin ""
-		)
-		(pin ""
-		)
-		(instances
-			(project ""
-				(path "/91e6286f-2f5f-4c12-b8bc-a46dfa772353"
-					(reference "S2")
-					(unit 1)
-				)
