File: source/cucabot/cucabot-plataforma-electric/cucabot-plataforma-electric.kicad_sch (KiCad schematic)
At the start: 20 parts, among them M1 motor, M2 motor, X1 borna_6x2

Commit message: 24/04/2026 Update
Parts:
- removed S2: selector_pack, symbol simbolos:selector_pack
- removed S2: selector, symbol electric-simbolos:selector
Connections:
- net at S1.: now also X1.
- net at X1.: no longer S1.
- net at X2.: now also V1., V2.; no longer S1.
- net at X3.: now also V2.
- net at X5.: no longer X6.
- new net: V1., V2., X1.
- new net: S1., X1.
- new net: M1., M2., X4.
- new net: S1., X2.
- new net: M1. (-), M2. (-), X1.
- now unconnected: X1., X1., X1., X1., X1., X1.
Other:
- note added: "PLATAFORMA UNIVERSAL CUCABOT"
- note removed: "NA"
- note removed: "NC"
- note removed: "ROBOT CUCABOT CERO"
- title: ROBOT CUCABOT CERO. ESQUEMAS ELÉCTRICOS -> ROBOT CUCABOT. PLATAFORMA UNIVERSAL
