File: source/cucabot/cucabot-pegatortas-electric/cucabot-pegatortas-electric.kicad_sch (KiCad schematic)
At the start: 20 parts, among them M1 motor, M2 motor, X1 borna_6x2

Commit message: 25/04/2026 Update
Parts:
- added S3: selector, symbol electric-simbolos:selector
- added S3: selector_pack, symbol simbolos:selector_pack
Connections:
- net at V2., X1.: no longer V1.
- net at S1.: now also X1.
- net at X2.: now also V1., V2.; no longer S1.
- net at X3.: now also V2.; no longer S2.
- net at S2., X5.: no longer X6.
- new net: V1., V2., X1.
- new net: S1., X1.
- new net: M1., M2., X4.
- new net: S1., X2.
- new net: S2., S3., X3.
- new net: S2., S3., X1. (x3)
- new net: S3., X6.
- new net: M1. (-), M2. (-), X1.
- new net: S3., X1.
Other:
- note added: "ANTENA DERECHA"
- note added: "ANTENA IZQUIERDA"
- note added: "ROBOT CUCABOT PEGATORTAS"
- note removed: "ROBOT CUCABOT MURÓFILO"
- title: ROBOT CUCABOT MURÓFILO. ESQUEMAS ELÉCTRICOS -> ROBOT CUCABOT PEGATORTAS. ESQUEMAS ELÉCTRICOS
- moved on the sheet: S2
