File: source/cucabot/cucabot-murofilo-electric/cucabot-murofilo-electric.kicad_sch (KiCad schematic)
At the start: 20 parts, among them M1 motor, M2 motor, X1 borna_6x2

Commit message: 25/04/2026 Update
Connections:
- net at S1.: now also X1.
- net at X1.: no longer S1.
- net at X2.: now also V1., V2.; no longer S1.
- net at X3.: now also V2.; no longer S2.
- new net: V1., V2., X1.
- new net: S1., X1.
- new net: M1., M2., X4.
- new net: S1., X2.
- new net: M1. (-), M2. (-), X1.
- new net: S2., X1. (x2)
- new net: S2., X5.
- new net: S2., X6.
- now unconnected: X1., X1., X1., X1., X1.
Changed lines of the file:
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@@
 	(text "NA"
 		(exclude_from_sim no)
-		(at 141.478 70.358 0)
+		(at 130.048 70.358 0)
 		(effects
 			(font
@@
 	(text "NC"
 		(exclude_from_sim no)
-		(at 141.732 57.404 0)
+		(at 130.048 57.15 0)
 		(effects
 			(font
@@
 	)
 	(junction
-		(at 104.14 212.09)
-		(diameter 0)
-		(color 0 0 0 0)
-	)
-	(junction
 		(at 96.52 207.01)
 		(diameter 0)
@@
 		(color 0 0 0 0)
 	)
-	(junction
-		(at 119.38 53.34)
-		(diameter 0)
-		(color 0 0 0 0)
-	)
 	(no_connect
 		(at 123.19 184.15)
@@
 	(wire
 		(pts
-			(xy 121.92 73.66) (xy 121.92 55.88)
-		)
-		(stroke
-			(width 0)
-			(type default)
-		)
-	)
-	(wire
-		(pts
 			(xy 85.09 66.04) (xy 85.09 73.66)
 		)
@@
 	(wire
 		(pts
-			(xy 106.68 214.63) (xy 106.68 217.17)
-		)
-		(stroke
-			(width 0)
-			(type default)
-		)
-	)
-	(wire
-		(pts
 			(xy 97.79 53.34) (xy 114.3 53.34)
 		)
@@
 	(wire
 		(pts
-			(xy 104.14 217.17) (xy 106.68 217.17)
+			(xy 127 67.31) (xy 129.54 67.31)
 		)
 		(stroke
@@
 	(wire
 		(pts
+			(xy 119.38 73.66) (xy 127 73.66)
+		)
+		(stroke
+			(width 0)
+			(type default)
+		)
+	)
+	(wire
+		(pts
 			(xy 83.82 212.09) (xy 96.52 212.09)
 		)
@@
 	(wire
 		(pts
-			(xy 137.16 88.9) (xy 146.05 88.9)
+			(xy 119.38 53.34) (xy 127 53.34)
 		)
 		(stroke
@@
 	(wire
 		(pts
-			(xy 119.38 53.34) (xy 124.46 53.34)
+			(xy 104.14 217.17) (xy 144.78 217.17)
 		)
 		(stroke
@@
 	(wire
 		(pts
-			(xy 146.05 67.31) (xy 146.05 88.9)
-		)
-		(stroke
-			(width 0)
-			(type default)
-		)
-	)
-	(wire
-		(pts
 			(xy 87.63 176.53) (xy 87.63 191.77)
 		)
@@
 	(wire
 		(pts
+			(xy 127 59.69) (xy 129.54 59.69)
+		)
+		(stroke
+			(width 0)
+			(type default)
+		)
+	)
+	(wire
+		(pts
 			(xy 44.45 46.99) (xy 44.45 39.37)
 		)
@@
 	(wire
 		(pts
-			(xy 127 63.5) (xy 127 55.88)
-		)
-		(stroke
-			(width 0)
-			(type default)
-		)
-	)
-	(wire
-		(pts
 			(xy 113.03 184.15) (xy 113.03 196.85)
 		)
@@
 		)
 	)
+	(wire
+		(pts
+			(xy 142.24 63.5) (xy 146.05 63.5)
+		)
+		(stroke
+			(width 0)
+			(type default)
+		)
+	)
 	(polyline
 		(pts
@@
 	(wire
 		(pts
+			(xy 104.14 191.77) (xy 149.86 191.77)
+		)
+		(stroke
+			(width 0)
+			(type default)
+		)
+	)
+	(wire
+		(pts
 			(xy 85.09 60.96) (xy 85.09 53.34)
 		)
@@
 		)
 	)
-	(wire
-		(pts
-			(xy 119.38 73.66) (xy 121.92 73.66)
-		)
-		(stroke
-			(width 0)
-			(type default)
-		)
-	)
-	(wire
-		(pts
-			(xy 127 55.88) (xy 124.46 53.34)
-		)
-		(stroke
-			(width 0)
-			(type default)
-		)
-	)
 	(polyline
 		(pts
@@
 	(wire
 		(pts
-			(xy 127 63.5) (xy 129.54 63.5)
-		)
-		(stroke
-			(width 0)
-			(type default)
-		)
-	)
-	(wire
-		(pts
 			(xy 85.09 53.34) (xy 87.63 53.34)
+		)
+		(stroke
+			(width 0)
+			(type default)
+		)
+	)
+	(wire
+		(pts
+			(xy 127 67.31) (xy 127 73.66)
 		)
 		(stroke
@@
 	(wire
 		(pts
-			(xy 142.24 67.31) (xy 146.05 67.31)
-		)
-		(stroke
-			(width 0)
-			(type default)
-		)
-	)
-	(wire
-		(pts
 			(xy 44.45 60.96) (xy 44.45 54.61)
 		)
@@
 	(wire
 		(pts
+			(xy 149.86 184.15) (xy 149.86 191.77)
+		)
+		(stroke
+			(width 0)
+			(type default)
+		)
+	)
+	(wire
+		(pts
 			(xy 82.55 63.5) (xy 85.09 66.04)
 		)
@@
 	(wire
 		(pts
-			(xy 104.14 212.09) (xy 106.68 214.63)
-		)
-		(stroke
-			(width 0)
-			(type default)
-		)
-	)
-	(wire
-		(pts
 			(xy 83.82 195.58) (xy 95.25 195.58)
 		)
@@
 	(wire
 		(pts
-			(xy 121.92 55.88) (xy 119.38 53.34)
+			(xy 127 53.34) (xy 127 59.69)
 		)
 		(stroke
@@
 	(wire
 		(pts
+			(xy 146.05 39.37) (xy 146.05 63.5)
+		)
+		(stroke
+			(width 0)
+			(type default)
+		)
+	)
+	(wire
+		(pts
 			(xy 52.07 63.5) (xy 59.69 63.5)
 		)
@@
 	(wire
 		(pts
-			(xy 142.24 59.69) (xy 146.05 59.69)
-		)
-		(stroke
-			(width 0)
-			(type default)
-		)
-	)
-	(wire
-		(pts
 			(xy 96.52 196.85) (xy 95.25 195.58)
 		)
@@
 	(wire
 		(pts
-			(xy 104.14 212.09) (xy 149.86 212.09)
-		)
-		(stroke
-			(width 0)
-			(type default)
-		)
-	)
-	(wire
-		(pts
 			(xy 44.45 88.9) (xy 132.08 88.9)
 		)
@@
 		)
 	)
-	(wire
-		(pts
-			(xy 146.05 39.37) (xy 146.05 59.69)
-		)
-		(stroke
-			(width 0)
-			(type default)
-		)
-	)
 	(polyline
 		(pts
@@
 	(wire
 		(pts
-			(xy 144.78 184.15) (xy 144.78 201.93)
+			(xy 104.14 212.09) (xy 139.7 212.09)
+		)
+		(stroke
+			(width 0)
+			(type default)
+		)
+	)
+	(wire
+		(pts
+			(xy 144.78 184.15) (xy 144.78 217.17)
 		)
 		(stroke
@@
 	(wire
 		(pts
-			(xy 104.14 191.77) (xy 139.7 191.77)
-		)
-		(stroke
-			(width 0)
-			(type default)
-		)
-	)
-	(wire
-		(pts
-			(xy 149.86 184.15) (xy 149.86 212.09)
-		)
-		(stroke
-			(width 0)
-			(type default)
-		)
-	)
-	(wire
-		(pts
 			(xy 78.74 198.12) (xy 95.25 198.12)
 		)
@@
 		)
 	)
-	(wire
-		(pts
-			(xy 139.7 184.15) (xy 139.7 191.77)
-		)
-		(stroke
-			(width 0)
-			(type default)
-		)
-	)
-	(wire
-		(pts
-			(xy 104.14 201.93) (xy 144.78 201.93)
-		)
-		(stroke
-			(width 0)
-			(type default)
-		)
-	)
 	(polyline
 		(pts
@@
 		(pts
 			(xy 64.77 201.93) (xy 96.52 201.93)
+		)
+		(stroke
+			(width 0)
+			(type default)
+		)
+	)
+	(wire
+		(pts
+			(xy 139.7 184.15) (xy 139.7 212.09)
 		)
 		(stroke
@@
 	(symbol
 		(lib_id "electric-simbolos:selector")
-		(at 129.54 63.5 0)
+		(at 142.24 63.5 0)
+		(mirror y)
 		(unit 1)
 		(exclude_from_sim no)
@@
 		(on_board yes)
 		(dnp no)
-		(fields_autoplaced yes)
 		(property "Reference" "S2"
 			(at 135.89 55.88 0)
@@
 		)
 		(property "Value" "selector"
-			(at 129.54 64.77 0)
+			(at 142.24 64.77 0)
 			(effects
 				(font
@@
 		)
 		(property "Footprint" ""
-			(at 137.16 67.31 0)
+			(at 134.62 67.31 0)
 			(effects
 				(font
@@
 		)
 		(property "Datasheet" ""
-			(at 137.16 67.31 0)
+			(at 134.62 67.31 0)
 			(effects
 				(font
@@
 		)
 		(property "Description" ""
-			(at 129.54 63.5 0)
-			(effects
-				(font
+			(at 142.24 63.5 0)
+			(effects
+				(font

Commit message: 27/04/2026 Update
Connections:
- net at S1.: now also X1.
- net at X1.: no longer S1.
- net at X2.: now also V1., V2.; no longer S1.
- net at X3.: now also V2.
- new net: V1., V2., X1.
- new net: S1., X1.
- new net: M1., M2., X4.
- new net: S2., X1. (x2)
- new net: S1., X2.
- new net: M1. (-), M2. (-), X1.
- now unconnected: X1., X1., X1., X1., X1.
Other:
- note added: "ANTENA"
Changed lines of the file:
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@@
+		)
+	)
+	(text "ANTENA"
+		(exclude_from_sim no)
+		(at 136.652 67.818 0)
+		(effects
+			(font
+				(size 1.905 1.905)
+			)
+			(justify left)
 		)
 	)
@@
 	)
 	(symbol
+		(lib_name "selector_pack_2")
+		(lib_id "simbolos:selector_pack")
+		(at 139.7 184.15 0)
+		(unit 1)
+		(exclude_from_sim no)
+		(in_bom yes)
+		(on_board yes)
+		(dnp no)
+		(property "Reference" "S2"
+			(at 147.574 175.006 0)
+			(effects
+				(font
+					(size 2.54 2.54)
+				)
+				(justify left)
+			)
+		)
+		(property "Value" "selector_pack"
+			(at 144.78 179.07 0)
+			(effects
+				(font
+					(size 1.27 1.27)
+				)
+				(hide yes)
+			)
+		)
+		(property "Footprint" ""
+			(at 147.32 187.96 0)
+			(effects
+				(font
+					(size 1.27 1.27)
+				)
+				(hide yes)
+			)
+		)
+		(property "Datasheet" ""
+			(at 147.32 187.96 0)
+			(effects
+				(font
+					(size 1.27 1.27)
+				)
+				(hide yes)
+			)
+		)
+		(property "Description" ""
+			(at 139.7 184.15 0)
+			(effects
+				(font
+					(size 1.27 1.27)
+				)
+			)
+		)
+		(pin ""
+		)
+		(pin ""
+		)
+		(pin ""
+		)
+		(instances
+			(project ""
+				(path "/91e6286f-2f5f-4c12-b8bc-a46dfa772353"
+					(reference "S2")
+					(unit 1)
+				)
+			)
+		)
+	)
+	(symbol
 		(lib_name "motor_1")
 		(lib_id "electric-simbolos:motor")
@@
 					(unit 1)
 				)
-			)
-		)
-	)
-	(symbol
-		(lib_name "selector_pack_1")
-		(lib_id "simbolos:selector_pack")
-		(at 139.7 184.15 0)
-		(unit 1)
-		(exclude_from_sim no)
-		(in_bom yes)
-		(on_board yes)
-		(dnp no)
-		(property "Reference" "S2"
-			(at 147.32 174.752 0)
-			(effects
-				(font
-					(size 2.54 2.54)
-				)
-				(justify left)
-			)
-		)
-		(property "Value" "selector_pack"
-			(at 144.78 179.07 0)
-			(effects
-				(font
-					(size 1.27 1.27)
-				)
-				(hide yes)
-			)
-		)
-		(property "Footprint" ""
-			(at 147.32 187.96 0)
-			(effects
-				(font
-					(size 1.27 1.27)
-				)
-				(hide yes)
-			)
-		)
-		(property "Datasheet" ""
-			(at 147.32 187.96 0)
-			(effects
-				(font
-					(size 1.27 1.27)
-				)
-				(hide yes)
-			)
-		)
-		(property "Description" ""
-			(at 139.7 184.15 0)
-			(effects
-				(font
-					(size 1.27 1.27)
-				)
-			)
-		)
-		(pin ""
-		)
-		(pin ""
-		)
-		(pin ""
-		)
-		(instances
-			(project "cucabot-murofilo-electric"
-				(path "/91e6286f-2f5f-4c12-b8bc-a46dfa772353"
-					(reference "S2")
-					(unit 1)
-				)
